File: 75-PCB.kicad_pcb (KiCad board)
At the start: 2 copper layers, 315.1 x 125.4 mm, 323 parts, among them J1 AVR-ISP-6, Q1 2N7002, SW1 SW_Push, U1 AT90USB1286-AU, U2 PRTR5V0U2X, Y1 16MHz

Commit message: Created duplex matrix for switches and switched MCU to ATMega32U4
Parts:
- U1: value AT90USB1286-AU -> ATmega32U4-AU; footprint Package_QFP:TQFP-64_14x14mm_P0.8mm -> Package_QFP:TQFP-44_10x10mm_P0.8mm
- moved C6 79.9 mm to (348.5, -218.4), turned to 90 degrees
- moved C4 75.0 mm to (363.5, -196.7), turned to 270 degrees
- moved C1 73.8 mm to (351.6, -182.6), turned to 270 degrees
- moved U1 73.3 mm to (352.4, -201.6)
- moved Y1 73.3 mm to (353.2, -186.5)
- moved C2 72.3 mm to (354.8, -182.6), turned to 270 degrees
- moved R4 67.7 mm to (333.2, -206.4), turned to 0 degrees
- moved C3 62.2 mm to (336.6, -215.2)
- moved C5 40.0 mm to (330.9, -194.5), turned to 180 degrees
- moved J1 32.5 mm to (283.4, -166.7), turned to 90 degrees
- moved MX_BCKSP2 19.1 mm to (268.3, -205.6)
- moved MX_BCKSP3 19.1 mm to (249.2, -205.6)
- moved Q1 17.2 mm to (286.5, -172.2)
- moved R11 17.2 mm to (283.4, -172.2)
- moved R10 17.2 mm to (281.0, -172.2)
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- renumbered D37 to D36, D38 to D37, D39 to D38, D40 to D39, D41 to D40, D36 to D41, D43 to D42, D44 to D43, D45 to D44, D46 to D45, D47 to D46, D48 to D47, D49 to D48, D50 to D49, D51 to D50, D52 to D51, D42 to D52, D54 to D53, D55 to D54, D56 to D55, D57 to D56, D58 to D57, D53 to D58, D60 to D59, D61 to D60, D62 to D61, D63 to D62, D64 to D63, D59 to D64, D66 to D65, D67 to D66, D68 to D67, D69 to D68, D70 to D69, D65 to D70, D75 to D74, D79 to D75, D80 to D79, D74 to D80, R13 to R12, R14 to R13, R15 to R14, R16 to R15, R17 to R16, R18 to R17, R19 to R18, R20 to R19, R21 to R20, R22 to R21, R23 to R22, R24 to R23, R25 to R24, R26 to R25, R27 to R26, R28 to R27, R29 to R28, R30 to R29, R31 to R30, R32 to R31, R33 to R32, R34 to R33, R35 to R34, R36 to R35, R37 to R36, R38 to R37, R39 to R38, R40 to R39, R41 to R40, R42 to R41, R43 to R42, R44 to R43, R45 to R44, R46 to R45, R48 to R46, R49 to R47, R50 to R48, R51 to R49, R52 to R50, R47 to R51, R54 to R52, R55 to R53, R56 to R54, R57 to R55, R58 to R56, R59 to R57, R60 to R58, R61 to R59, R62 to R60, R63 to R61, R53 to R62, R65 to R63, R66 to R64, R67 to R65, R68 to R66, R69 to R67, R64 to R68, R71 to R69, R72 to R70, R73 to R71, R74 to R72, R75 to R73, R70 to R74, R77 to R75, R78 to R76, R79 to R77, R80 to R78, R81 to R79, R76 to R80, R82 to R81, R83 to R82, R84 to R83, R86 to R84, R90 to R85, R87 to R86, R88 to R87, R89 to R88, R91 to R89, R85 to R90, R92 to R91, R93 to R92, R94 to R93, R95 to R94, R96 to R95, R97 to R96, R98 to R97, R99 to R98
Connections:
- net RGBLED renamed Net-(LED9-Pad4)
- D10 pad 1: ROW2 -> ROW5
- D11 pad 1: ROW3 -> ROW6
- D12 pad 1: ROW4 -> COL9
- D13 pad 1: ROW5 -> COL10
- D15 pad 1: ROW1 -> ROW3
- D16 pad 1: ROW2 -> ROW4
- D17 pad 1: ROW3 -> ROW7
- D18 pad 1: ROW4 -> COL8
- D19 pad 1: ROW5 -> COL11
- D20 pad 1: ROW0 -> ROW1
- D21 pad 1: ROW1 -> ROW2
- D22 pad 1: ROW2 -> ROW5
- D23 pad 1: ROW3 -> ROW6
- D24 pad 1: ROW4 -> COL9
- D26 pad 1: ROW1 -> ROW3
- D27 pad 1: ROW2 -> ROW4
- D28 pad 1: ROW3 -> ROW7
- D29 pad 1: ROW4 -> COL8
- D3 pad 1: ROW1 -> ROW3
- D30 pad 1: ROW5 -> COL10
- D31 pad 1: ROW0 -> ROW1
- D32 pad 1: ROW1 -> ROW2
- D33 pad 1: ROW2 -> ROW5
- D34 pad 1: ROW3 -> ROW6
- D35 pad 1: ROW4 -> COL9
- D37 pad 1: ROW1 -> ROW3
- D38 pad 1: ROW2 -> ROW4
- D39 pad 1: ROW3 -> ROW7
- D4 pad 1: ROW2 -> ROW4
- D40 pad 1: ROW4 -> COL8
- D41 pad 1: ROW5 -> COL11
- D42 pad 1: ROW0 -> ROW1
- D43 pad 1: ROW1 -> ROW2
- D44 pad 1: ROW2 -> ROW5
- D45 pad 1: ROW3 -> ROW6
- D46 pad 1: ROW4 -> COL9
- D48 pad 1: ROW1 -> ROW3
- D49 pad 1: ROW2 -> ROW4
- D5 pad 1: ROW3 -> ROW7
- D50 pad 1: ROW3 -> ROW7
- D51 pad 1: ROW4 -> COL8
- D52 pad 1: ROW5 -> COL10
- D53 pad 1: ROW0 -> ROW1
- D54 pad 1: ROW1 -> ROW2
- D55 pad 1: ROW2 -> ROW5
- D56 pad 1: ROW3 -> ROW6
- D57 pad 1: ROW4 -> COL9
- D58 pad 1: ROW5 -> COL11
- D6 pad 1: ROW4 -> COL8
- D60 pad 1: ROW1 -> ROW3
- D61 pad 1: ROW2 -> ROW4
- D62 pad 1: ROW3 -> ROW7
- D63 pad 1: ROW4 -> COL8
- D64 pad 1: ROW5 -> COL10
- D65 pad 1: ROW0 -> ROW1
- D66 pad 1: ROW1 -> ROW2
- D67 pad 1: ROW2 -> ROW5
- D68 pad 1: ROW3 -> ROW6
- D69 pad 1: ROW4 -> COL9
- D7 pad 1: ROW5 -> COL11
- D70 pad 1: ROW5 -> COL11
- D72 pad 1: ROW1 -> ROW3
- D73 pad 1: ROW2 -> ROW4
- D74 pad 1: ROW4 -> COL8
- D75 pad 1: ROW5 -> COL10
- D76 pad 1: ROW0 -> ROW1
- D77 pad 1: ROW1 -> ROW2
- D78 pad 1: ROW2 -> ROW5
- D79 pad 1: ROW1 -> ROW3
- D8 pad 1: ROW0 -> ROW1
- D80 pad 1: ROW3 -> ROW7
- D81 pad 1: ROW4 -> COL9
- D82 pad 1: ROW5 -> COL11
- D84 pad 1: ROW1 -> ROW2
- D85 pad 1: ROW2 -> ROW4
- D89 pad 1: ROW3 -> ROW6
- D9 pad 1: ROW1 -> ROW2
- D90 pad 1: ROW4 -> COL8
- D91 pad 1: ROW5 -> COL10
- LED2 pad 2: Net-(LED1-Pad4) -> Net-(LED2-Pad2)
- LED3 pad 2: Net-(LED2-Pad4) -> Net-(LED3-Pad2)
- LED4 pad 1: +5V -> Net-(LED4-Pad1)
- LED4 pad 2: Net-(LED3-Pad4) -> Net-(LED4-Pad2)
- LED5 pad 2: Net-(LED4-Pad4) -> Net-(LED5-Pad2)
- LED6 pad 2: Net-(LED5-Pad4) -> Net-(LED6-Pad2)
- LED7 pad 2: Net-(LED6-Pad4) -> Net-(LED7-Pad2)
- LED8 pad 2: Net-(LED7-Pad4) -> Net-(LED8-Pad2)
- LED9 pad 2: Net-(LED8-Pad4) -> Net-(LED9-Pad2)
- MX_#0 pad 1: COL10 -> COL5
- MX_#1 pad 1: COL1 -> COL0
- MX_#2 pad 1: COL2 -> COL1
- MX_#3 pad 1: COL3 -> COL1
- MX_#3 pad 3: +5V -> Net-(MX_#3-Pad3)
- MX_#4 pad 1: COL4 -> COL2
- MX_#5 pad 1: COL5 -> COL2
- MX_#5 pad 3: +5V -> Net-(MX_#5-Pad3)
- MX_#6 pad 1: COL6 -> COL3
- MX_#7 pad 1: COL7 -> COL3
- MX_#7 pad 3: +5V -> Net-(MX_#7-Pad3)
- MX_#8 pad 1: COL8 -> COL4
- MX_#9 pad 1: COL9 -> COL4
- MX_'1 pad 1: COL11 -> COL5
- MX_,1 pad 1: COL9 -> COL4
- MX_-1 pad 1: COL11 -> COL5
- MX_.1 pad 1: COL10 -> COL5
- MX_/1 pad 1: COL11 -> COL5
- MX_;1 pad 1: COL10 -> COL5
- MX_=1 pad 1: COL12 -> COL6
- MX_A1 pad 1: COL1 -> COL0
- MX_B1 pad 1: COL6 -> COL3
- MX_BCKSP1 pad 1: COL13 -> COL6
- MX_BCKSP2 pad 1: COL13 -> COL6
- MX_BCKSP3 pad 1: COL14 -> COL7
- MX_C1 pad 1: COL4 -> COL2
- MX_D1 pad 1: COL3 -> COL1
- MX_D1 pad 3: +5V -> Net-(MX_D1-Pad3)
- MX_DEL1 pad 1: COL15 -> COL7
- MX_DOWN1 pad 1: COL14 -> COL7
- MX_E1 pad 1: COL3 -> COL1
- MX_E1 pad 3: +5V -> Net-(MX_E1-Pad3)
- MX_END1 pad 1: COL15 -> COL7
- MX_ENTER1 pad 1: COL14 -> COL7
- MX_ENTER2 pad 1: COL14 -> Net-(MX_ENTER2-Pad1)
- MX_ENTER2 pad 3: +5V -> Net-(MX_ENTER2-Pad3)
- MX_F#1 pad 1: COL1 -> COL0
- MX_F#10 pad 1: COL10 -> COL5
- MX_F#11 pad 1: COL11 -> COL5
- MX_F#12 pad 1: COL12 -> COL6
- MX_F#2 pad 1: COL2 -> COL1
- MX_F#3 pad 1: COL3 -> COL1
- MX_F#3 pad 3: +5V -> Net-(MX_F#3-Pad3)
- MX_F#4 pad 1: COL4 -> COL2
- MX_F#5 pad 1: COL5 -> COL2
- MX_F#5 pad 3: +5V -> Net-(MX_F#5-Pad3)
- MX_F#6 pad 1: COL6 -> COL3
- MX_F#7 pad 1: COL7 -> COL3
- MX_F#7 pad 3: +5V -> Net-(MX_F#7-Pad3)
- MX_F#8 pad 1: COL8 -> COL4
- MX_F#9 pad 1: COL9 -> COL4
- MX_F1 pad 1: COL4 -> COL2
- MX_G1 pad 1: COL5 -> COL2
- MX_G1 pad 3: +5V -> Net-(MX_G1-Pad3)
- MX_H1 pad 1: COL6 -> COL3
- MX_HOME1 pad 1: COL15 -> COL7
- MX_I1 pad 1: COL8 -> COL4
- MX_J1 pad 1: COL7 -> COL3
- MX_J1 pad 3: +5V -> Net-(MX_J1-Pad3)
- MX_K1 pad 1: COL8 -> COL4
- MX_L1 pad 1: COL9 -> COL4
- MX_LALT1 pad 1: COL2 -> COL1
- MX_LALT2 pad 1: COL2 -> COL1
- MX_LALT3 pad 1: COL2 -> COL1
- MX_LALT3 pad 4: Net-(MX_LALT3-Pad4) -> Net-(MX_LALT1-Pad4)
- MX_LEFT1 pad 1: COL12 -> COL6
- MX_LSHIFT3 pad 1: COL1 -> COL0
- MX_LWIN1 pad 1: COL1 -> COL0
- MX_LWIN1 pad 4: Net-(MX_LALT3-Pad4) -> Net-(MX_LWIN1-Pad4)
- MX_LWIN2 pad 1: COL1 -> COL0
- MX_LWIN2 pad 4: Net-(MX_LALT3-Pad4) -> Net-(MX_LWIN1-Pad4)
- MX_M1 pad 1: COL8 -> COL4
- MX_N1 pad 1: COL7 -> COL3
- MX_N1 pad 3: +5V -> Net-(MX_N1-Pad3)
- MX_O1 pad 1: COL9 -> COL4
- MX_P1 pad 1: COL10 -> COL5
- MX_PAUSE1 pad 1: COL13 -> COL6
- MX_PGDN1 pad 1: COL15 -> COL7
- MX_PGUP1 pad 1: COL15 -> COL7
- MX_Q1 pad 1: COL1 -> COL0
- MX_R1 pad 1: COL4 -> COL2
- MX_RALT1 pad 1: COL9 -> COL4
- MX_RALT2 pad 1: COL9 -> COL4
- MX_RCTRL1 pad 1: COL11 -> COL5
- MX_RCTRL2 pad 1: COL11 -> COL5
- MX_RIGHT1 pad 1: COL15 -> COL7
- MX_RSHIFT1 pad 1: COL12 -> COL6
- MX_RWIN1 pad 1: COL10 -> COL5
- MX_S1 pad 1: COL2 -> COL1
- MX_SPACE1 pad 1: COL6 -> COL3
- MX_SPACE2 pad 1: COL6 -> COL3
- MX_SPACE3 pad 1: COL6 -> COL3
- MX_SPACE4 pad 1: COL6 -> COL3
- MX_SPACE5 pad 1: COL4 -> COL2
- MX_SPACE6 pad 1: COL8 -> COL4
- MX_T1 pad 1: COL5 -> COL2
- MX_T1 pad 3: +5V -> Net-(MX_T1-Pad3)
- MX_U1 pad 1: COL7 -> COL3
- MX_U1 pad 3: +5V -> Net-(MX_U1-Pad3)
- MX_UP1 pad 1: COL14 -> COL7
- MX_V1 pad 1: COL5 -> COL2
- MX_V1 pad 3: +5V -> Net-(MX_V1-Pad3)
- MX_W1 pad 1: COL2 -> COL1
- MX_X1 pad 1: COL3 -> COL1
- MX_X1 pad 3: +5V -> Net-(MX_X1-Pad3)
- MX_Y1 pad 1: COL6 -> COL3
- MX_Z1 pad 1: COL2 -> COL1
- MX_[1 pad 1: COL11 -> COL5
- MX_\1 pad 1: COL13 -> COL6
- MX_\2 pad 1: COL13 -> COL6
- MX_]1 pad 1: COL12 -> COL6
- R23 pad 1: Net-(MX_LALT3-Pad4) -> Net-(MX_LWIN1-Pad4)
- R4 pad 1: Net-(R4-Pad1) -> GND
- R4 pad 2: GND -> Net-(R4-Pad2)
- U1 pad 11: SCK -> Net-(U1-Pad11)
- U1 pad 12: MOSI -> LEDMOS
- U1 pad 13: MISO -> RESET
- U1 pad 14: Net-(U1-Pad14) -> +5V
- U1 pad 15: Net-(U1-Pad15) -> GND
- U1 pad 16: Net-(U1-Pad16) -> Net-(C2-Pad1)
- U1 pad 17: LEDMOS -> Net-(C1-Pad1)
- U1 pad 2: Net-(U1-Pad2) -> +5V
- U1 pad 20: RESET -> Net-(U1-Pad20)
- U1 pad 21: +5V -> Net-(U1-Pad21)
- U1 pad 22: GND -> Net-(U1-Pad22)
- U1 pad 23: Net-(C2-Pad1) -> GND
- U1 pad 24: Net-(C1-Pad1) -> +5V
- U1 pad 3: +5V -> D-
- U1 pad 33: Net-(U1-Pad33) -> Net-(R4-Pad2)
- U1 pad 34: Net-(U1-Pad34) -> +5V
- U1 pad 35: Net-(U1-Pad35) -> GND
- U1 pad 4: D- -> D+
- U1 pad 43: Net-(R4-Pad1) -> GND
- U1 pad 44: Net-(U1-Pad44) -> +5V
- U1 pad 5: D+ -> GND
- U1 pad 6: GND -> Net-(C7-Pad1)
- U1 pad 7: Net-(C7-Pad1) -> +5V
- U1 pad 8: +5V -> Net-(U1-Pad8)
Routing:
- net +5V: track 2514.4 -> 0.00 mm, vias 24 -> 0
- net LEDGND: track 1836.5 -> 0.00 mm, vias 13 -> 0
- net ROW3: track 301.4 -> 0.00 mm, vias 4 -> 0
- net ROW4: track 299.5 -> 0.00 mm
- net ROW0: track 294.4 -> 0.00 mm, vias 2 -> 0
- net ROW1: track 292.5 -> 0.00 mm, vias 2 -> 0
- net ROW5: track 288.8 -> 0.00 mm
- net ROW2: track 287.4 -> 0.00 mm, vias 4 -> 0
- net GND: track 245.9 -> 0.00 mm, vias 5 -> 0
- net COL6: track 130.6 -> 0.00 mm
- net COL2: track 129.3 -> 0.00 mm
- net COL9: track 125.4 -> 0.00 mm
- net COL10: track 120.6 -> 0.00 mm
- net COL11: track 119.9 -> 0.00 mm
- net COL0: track 117.0 -> 0.00 mm
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