File: 75-PCB.kicad_pcb (KiCad board)
At the start: 2 copper layers, 315.1 x 125.4 mm, 323 parts, among them J1 AVR-ISP-6, Q1 2N7002, SW1 SW_Push, U1 ATmega32U4-AU, U2 PRTR5V0U2X, Y1 16MHz

Commit message: Finished USB and MCU traces
Parts:
- moved C6 87.9 mm to (273.7, -172.2), turned to 180 degrees
- moved U1 73.3 mm to (283.4, -177.0), turned to 270 degrees
- moved C4 71.3 mm to (293.7, -182.6), turned to 0 degrees
- moved R4 66.9 mm to (279.4, -166.7), turned to 90 degrees
- moved C3 65.8 mm to (277.0, -187.3)
- moved Y1 59.5 mm to (294.5, -177.0), turned to 90 degrees
- moved R5 58.2 mm to (346.1, -150.2)
- moved C2 56.5 mm to (298.4, -178.6), turned to 0 degrees
- moved J1 53.9 mm to (321.5, -204.8), turned to 0 degrees
- moved C1 53.7 mm to (298.4, -175.4), turned to 0 degrees
- moved C5 51.6 mm to (287.3, -166.7), turned to 90 degrees
- moved SW1 40.2 mm to (322.3, -170.7)
- moved R51 31.8 mm to (108.0, -123.8)
- moved R9 31.2 mm to (282.6, -187.3)
- moved R8 31.0 mm to (280.2, -187.3)
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Routing:
- net GND: track 0.00 -> 120.3 mm, vias 0 -> 2
- net +5V: track 0.00 -> 102.7 mm, vias 0 -> 8
- net Net-(R9-Pad2): track 0.00 -> 50.7 mm, vias 0 -> 1
- net Net-(R8-Pad2): track 0.00 -> 49.4 mm, vias 0 -> 2
- net VCC: track 0.00 -> 26.3 mm, vias 0 -> 1
- net Net-(C2-Pad1): track 0.00 -> 10.5 mm
- net Net-(C1-Pad1): track 0.00 -> 10.3 mm
- net Net-(R7-Pad2): track 0.00 -> 9.43 mm
- net Net-(R6-Pad2): track 0.00 -> 7.84 mm, vias 0 -> 1
- net D+: track 0.00 -> 4.19 mm
- net D-: track 0.00 -> 4.15 mm
- net Net-(R4-Pad2): track 0.00 -> 3.69 mm
- net Net-(D1-Pad2): track 0.00 -> 1.71 mm

Commit message: Finished column and row traces
Parts:
- moved R89 35.0 mm to (241.3, -200.0)
- moved R87 35.0 mm to (276.2, -197.8)
- moved D79 0.79 mm to (276.2, -202.4)
Connections:
- net COL10 renamed ROW10
- net COL11 renamed ROW11
- net COL8 renamed ROW8
- net COL9 renamed ROW9
- MX_#3 pad 3: Net-(MX_#3-Pad3) -> +5V
- MX_#5 pad 3: Net-(MX_#5-Pad3) -> +5V
- MX_#7 pad 3: Net-(MX_#7-Pad3) -> +5V
- MX_BCKSP1 pad 1: COL6 -> COL7
- MX_BCKSP1 pad 2: Net-(D77-Pad2) -> Net-(D79-Pad2)
- MX_BCKSP2 pad 1: COL6 -> COL7
- MX_BCKSP2 pad 2: Net-(D77-Pad2) -> Net-(D79-Pad2)
- MX_BCKSP3 pad 1: COL7 -> COL6
- MX_BCKSP3 pad 2: Net-(D79-Pad2) -> Net-(D77-Pad2)
- MX_D1 pad 3: Net-(MX_D1-Pad3) -> +5V
- MX_E1 pad 3: Net-(MX_E1-Pad3) -> +5V
- MX_ENTER1 pad 1: COL7 -> COL6
- MX_ENTER2 pad 1: Net-(MX_ENTER2-Pad1) -> COL6
- MX_ENTER2 pad 3: Net-(MX_ENTER2-Pad3) -> +5V
- MX_F#3 pad 3: Net-(MX_F#3-Pad3) -> +5V
- MX_F#5 pad 3: Net-(MX_F#5-Pad3) -> +5V
- MX_F#7 pad 3: Net-(MX_F#7-Pad3) -> +5V
- MX_G1 pad 3: Net-(MX_G1-Pad3) -> +5V
- MX_J1 pad 3: Net-(MX_J1-Pad3) -> +5V
- MX_N1 pad 3: Net-(MX_N1-Pad3) -> +5V
- MX_T1 pad 3: Net-(MX_T1-Pad3) -> +5V
- MX_U1 pad 3: Net-(MX_U1-Pad3) -> +5V
- MX_V1 pad 3: Net-(MX_V1-Pad3) -> +5V
- MX_X1 pad 3: Net-(MX_X1-Pad3) -> +5V
- R87 pad 1: Net-(MX_BCKSP1-Pad4) -> Net-(MX_BCKSP3-Pad4)
- R89 pad 1: Net-(MX_BCKSP3-Pad4) -> Net-(MX_BCKSP1-Pad4)
Routing:
- net +5V: track 102.7 -> 1745.7 mm
- net LEDGND: track 0.00 -> 1472.9 mm
- net ROW4: track 0.00 -> 294.5 mm, vias 0 -> 2
- net ROW8: track 0.00 -> 267.7 mm
- net ROW7: track 0.00 -> 264.8 mm
- net ROW0: track 0.00 -> 256.6 mm
- net ROW1: track 0.00 -> 249.7 mm
- net ROW3: track 0.00 -> 242.3 mm
- net COL5: track 0.00 -> 240.6 mm
- net COL4: track 0.00 -> 235.7 mm
- net ROW11: track 0.00 -> 233.0 mm
- net COL1: track 0.00 -> 229.7 mm
- net ROW10: track 0.00 -> 221.9 mm
- net COL0: track 0.00 -> 220.9 mm
- net COL3: track 0.00 -> 220.7 mm
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
Commit message: Updated underglow LED placement
Parts:
- moved LED2 2.38 mm to (-4.76, -195.3)
- moved LED1 2.38 mm to (-4.76, -157.2)
- moved C15 0.79 mm to (305.6, -191.3)
- moved C16 0.79 mm to (305.6, -153.2)
- moved LED8 0.79 mm to (304.0, -196.8)
- moved LED5 0.79 mm to (132.6, -231.0)
- moved LED7 0.79 mm to (261.1, -231.0)
- moved LED9 0.79 mm to (304.0, -158.8)
Changed lines of the file:
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@@
   )
   (module WS2812B:WS2812B (layer B.Cu)
-    (at 304.00625 -197.64375)
+    (at 304.00625 -196.85)
     (fp_text reference LED8 (at 0 4.572) (layer B.SilkS)
       (effects (font (size 1 1) (thickness 0.15)) (justify mirror))
@@
   )
   (module WS2812B:WS2812B (layer B.Cu)
-    (at 304.00625 -159.54375)
+    (at 304.00625 -158.75)
     (fp_text reference LED9 (at 0 4.572) (layer B.SilkS)
       (effects (font (size 1 1) (thickness 0.15)) (justify mirror))
@@
   )
   (module WS2812B:WS2812B (layer B.Cu)
-    (at 261.9375 -230.98125 90)
+    (at 261.14375 -230.98125 90)
     (fp_text reference LED7 (at 0 4.572 90) (layer B.SilkS)
       (effects (font (size 1 1) (thickness 0.15)) (justify mirror))
@@
   )
   (module WS2812B:WS2812B (layer B.Cu)
-    (at 133.35 -230.98125 90)
+    (at 132.55625 -230.98125 90)
     (fp_text reference LED5 (at 0 4.572 270) (layer B.SilkS)
       (effects (font (size 1 1) (thickness 0.15)) (justify mirror))
@@
   )
   (module WS2812B:WS2812B (layer B.Cu)
-    (at -4.7625 -197.64375 180)
+    (at -4.7625 -195.2625 180)
     (fp_text reference LED2 (at 0 4.572 180) (layer B.SilkS)
       (effects (font (size 1 1) (thickness 0.15)) (justify mirror))
@@
   )
   (module WS2812B:WS2812B (layer B.Cu)
-    (at -4.7625 -159.54375 180)
+    (at -4.7625 -157.1625 180)
     (fp_text reference LED1 (at 0 4.572 180) (layer B.SilkS)
       (effects (font (size 1 1) (thickness 0.15)) (justify mirror))
@@
   )
   (module Capacitor_SMD:C_0805_2012Metric (layer B.Cu)
-    (at 305.59375 -153.9875 270)
+    (at 305.59375 -153.19375 270)
     (descr "Capacitor SMD 0805 (2012 Metric), square (rectangular) end terminal, IPC_7351 nominal, (Body size source: https://docs.google.com/spreadsheets/d/1BsfQQcO9C6DZCsRaXUlFlo91Tg2WpOkGARC1WS5S8t0/edit?usp=sharing), generated with kicad-footprint-generator")
     (tags capacitor)
@@
   )
   (module Capacitor_SMD:C_0805_2012Metric (layer B.Cu)
-    (at 305.59375 -192.0875 270)
+    (at 305.59375 -191.29375 270)
     (descr "Capacitor SMD 0805 (2012 Metric), square (rectangular) end terminal, IPC_7351 nominal, (Body size source: https://docs.google.com/spreadsheets/d/1BsfQQcO9C6DZCsRaXUlFlo91Tg2WpOkGARC1WS5S8t0/edit?usp=sharing), generated with kicad-footprint-generator")
     (tags capacitor)

Commit message: Changed underglow LED model
Parts:
- removed LED1, LED2, LED3, LED4, LED5, LED6, LED7, LED8, LED9: WS2812B, WS2812B:WS2812B
- added C17: 0.1uF, Capacitor_SMD:C_0805_2012Metric, B.Cu at (240.5, -95.2)
- added C18: 0.1uF, Capacitor_SMD:C_0805_2012Metric, B.Cu at (247.5, -93.2)
- added C19: 0.1uF, Capacitor_SMD:C_0805_2012Metric, B.Cu at (240.5, -98.2)
- added C20: 0.1uF, Capacitor_SMD:C_0805_2012Metric, B.Cu at (254.5, -85.2)
- added C21: 0.1uF, Capacitor_SMD:C_0805_2012Metric, B.Cu at (247.5, -90.2)
- added RGB1: SK6812MINI, LED_SMD:LED_SK6812MINI_PLCC4_3.5x3.5mm_P1.75mm, B.Cu at (304.0, -158.8)
- added RGB10: SK6812MINI, LED_SMD:LED_SK6812MINI_PLCC4_3.5x3.5mm_P1.75mm, B.Cu at (13.5, -122.2)
- added RGB11: SK6812MINI, LED_SMD:LED_SK6812MINI_PLCC4_3.5x3.5mm_P1.75mm, B.Cu at (107.2, -122.2)
- added RGB12: SK6812MINI, LED_SMD:LED_SK6812MINI_PLCC4_3.5x3.5mm_P1.75mm, B.Cu at (177.8, -123.0)
- added RGB13: SK6812MINI, LED_SMD:LED_SK6812MINI_PLCC4_3.5x3.5mm_P1.75mm, B.Cu at (218.3, -123.0)
- added RGB14: SK6812MINI, LED_SMD:LED_SK6812MINI_PLCC4_3.5x3.5mm_P1.75mm, B.Cu at (284.2, -118.3)
- added RGB2: SK6812MINI, LED_SMD:LED_SK6812MINI_PLCC4_3.5x3.5mm_P1.75mm, B.Cu at (304.0, -196.8)
- added RGB3: SK6812MINI, LED_SMD:LED_SK6812MINI_PLCC4_3.5x3.5mm_P1.75mm, B.Cu at (261.1, -231.0)
- added RGB4: SK6812MINI, LED_SMD:LED_SK6812MINI_PLCC4_3.5x3.5mm_P1.75mm, B.Cu at (202.4, -231.0)
- added RGB5: SK6812MINI, LED_SMD:LED_SK6812MINI_PLCC4_3.5x3.5mm_P1.75mm, B.Cu at (132.6, -231.0)
- added RGB6: SK6812MINI, LED_SMD:LED_SK6812MINI_PLCC4_3.5x3.5mm_P1.75mm, B.Cu at (73.0, -231.0)
- added RGB7: SK6812MINI, LED_SMD:LED_SK6812MINI_PLCC4_3.5x3.5mm_P1.75mm, B.Cu at (11.1, -231.0)
- added RGB8: SK6812MINI, LED_SMD:LED_SK6812MINI_PLCC4_3.5x3.5mm_P1.75mm, B.Cu at (-4.76, -195.3)
- added RGB9: SK6812MINI, LED_SMD:LED_SK6812MINI_PLCC4_3.5x3.5mm_P1.75mm, B.Cu at (-4.76, -157.2)
- moved R5 55.7 mm to (290.5, -154.0), turned to 270 degrees
- moved SW1 43.7 mm to (283.4, -150.8)
- moved Q1 42.4 mm to (281.0, -155.6), turned to 180 degrees
- moved R11 39.0 mm to (284.2, -155.6), turned to 270 degrees
- moved J1 38.8 mm to (283.4, -197.6)
- moved R10 36.5 mm to (286.5, -155.6), turned to 270 degrees
- moved D36 15.9 mm to (117.5, -224.6)
- moved C13 2.38 mm to (-6.35, -200.8)
- moved C14 2.38 mm to (-6.35, -162.7)
- moved C10 0.79 mm to (138.1, -232.6)
- moved C12 0.79 mm to (266.7, -232.6)
- turned R1 to 0 degrees
- turned R2 to 0 degrees
- turned R3 to 0 degrees
Routing:
- net COL7: track 172.3 -> 113.2 mm
- net ROW4: track 294.5 -> 247.1 mm, vias 2 -> 0
- net Net-(U1-Pad25): track 0.00 -> 24.1 mm
- net Net-(U1-Pad26): track 0.00 -> 23.1 mm
- net Net-(U1-Pad27): track 0.00 -> 22.1 mm
- net Net-(U1-Pad28): track 0.00 -> 21.1 mm
- net Net-(U1-Pad29): track 0.00 -> 20.1 mm
- net Net-(U1-Pad30): track 0.00 -> 19.2 mm
- net Net-(U1-Pad31): track 0.00 -> 18.4 mm
- net Net-(U1-Pad32): track 0.00 -> 17.7 mm
- net GND: track 120.3 -> 137.6 mm
- net Net-(U1-Pad39): track 0.00 -> 16.9 mm
- net Net-(U1-Pad40): track 0.00 -> 15.9 mm
- net Net-(U1-Pad41): track 0.00 -> 14.9 mm
- net COL6: track 202.9 -> 217.4 mm
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
Commit message: Finished routing traces around underglow LEDs
Parts:
- J1: moved to B.Cu
- moved C15 308.0 mm to (-2.38, -195.3)
- moved C16 308.0 mm to (-2.38, -157.2)
- moved C8 294.4 mm to (301.6, -158.8), turned to 90 degrees
- moved C17 229.0 mm to (13.5, -125.4)
- moved C9 225.9 mm to (301.6, -196.8), turned to 90 degrees
- moved C18 144.0 mm to (107.2, -125.4)
- moved C12 134.2 mm to (132.6, -228.6), turned to 180 degrees
- moved C10 123.1 mm to (261.1, -228.6), turned to 180 degrees
- moved C13 84.1 mm to (73.0, -228.6), turned to 180 degrees
- moved C19 68.4 mm to (177.8, -125.4)
- moved C14 68.2 mm to (11.1, -228.6), turned to 180 degrees
- moved C20 54.2 mm to (218.3, -125.4)
- moved C21 48.1 mm to (284.2, -121.4)
- moved D41 34.9 mm to (142.9, -129.4)
- moved R51 34.9 mm to (142.9, -123.8)
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Routing:
- net +5V: track 1747.8 -> 1843.3 mm
- net GND: track 137.6 -> 208.9 mm
- net LEDGND: track 1472.9 -> 1522.1 mm
- net ROW11: track 233.0 -> 273.9 mm
- net Net-(MX_RWIN1-Pad4): track 6.48 -> 32.7 mm
- net Net-(D64-Pad2): track 6.18 -> 30.6 mm
- net ROW10: track 221.9 -> 242.1 mm
- net Net-(MX_RIGHT1-Pad4): track 9.88 -> 29.6 mm
- net Net-(D91-Pad2): track 11.9 -> 20.9 mm
- net Net-(D75-Pad2): track 6.82 -> 15.9 mm
- net Net-(D52-Pad2): track 6.82 -> 0.00 mm
- net Net-(D20-Pad2): track 6.82 -> 0.00 mm
- net Net-(MX_DOWN1-Pad4): track 7.27 -> 12.6 mm
- net Net-(D41-Pad2): track 30.9 -> 25.9 mm
- net Net-(D82-Pad2): track 6.82 -> 10.0 mm
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
Commit message: Added mounting holes
Parts:
- added H1: MountingHole, mounting_hole:mounting, F.Cu at (18.3, -186.5)
- added H2: MountingHole, mounting_hole:mounting, F.Cu at (120.7, -167.5)
- added H3: MountingHole, mounting_hole:mounting, F.Cu at (251.6, -186.5)
- moved R5 12.1 mm to (285.8, -142.9), turned to 90 degrees
- moved D34 7.14 mm to (119.1, -174.6)
- moved D4 7.14 mm to (14.3, -193.7)
- moved D73 5.56 mm to (247.7, -192.1)
- moved D78 5.56 mm to (250.8, -192.1)
Connections:
- net Net-(RGB1-Pad3) renamed RGBLED
- RGB11 pad 3: Net-(RGB11-Pad3) -> Net-(RGB10-Pad1)
- RGB12 pad 3: Net-(RGB12-Pad3) -> Net-(RGB11-Pad1)
- RGB13 pad 3: Net-(RGB13-Pad3) -> Net-(RGB12-Pad1)
- RGB14 pad 3: Net-(RGB14-Pad3) -> Net-(RGB13-Pad1)
- RGB2 pad 3: Net-(RGB2-Pad3) -> Net-(RGB1-Pad1)
- RGB3 pad 3: Net-(RGB3-Pad3) -> Net-(RGB2-Pad1)
- RGB4 pad 3: Net-(RGB4-Pad3) -> Net-(RGB3-Pad1)
- RGB5 pad 3: Net-(RGB5-Pad3) -> Net-(RGB4-Pad1)
- RGB6 pad 3: Net-(RGB6-Pad3) -> Net-(RGB5-Pad1)
- RGB7 pad 3: Net-(RGB7-Pad3) -> Net-(RGB6-Pad1)
- RGB8 pad 3: Net-(RGB8-Pad3) -> Net-(RGB7-Pad1)
- RGB9 pad 1: Net-(RGB9-Pad1) -> Net-(RGB10-Pad3)
- RGB9 pad 3: Net-(RGB9-Pad3) -> Net-(RGB8-Pad1)
Routing:
- net +5V: track 1843.3 -> 2019.3 mm
- net Net-(RGB10-Pad1): track 0.00 -> 91.6 mm
- net LEDGND: track 1522.1 -> 1605.0 mm, vias 0 -> 7
- net Net-(RGB11-Pad1): track 0.00 -> 68.6 mm
- net Net-(RGB2-Pad1): track 0.00 -> 67.5 mm, vias 0 -> 2
- net Net-(RGB4-Pad1): track 0.00 -> 67.1 mm
- net Net-(RGB13-Pad1): track 0.00 -> 65.3 mm
- net ROW9: track 196.2 -> 258.4 mm
- net Net-(RGB6-Pad1): track 0.00 -> 59.1 mm
- net Net-(RGB5-Pad1): track 0.00 -> 56.8 mm
- net Net-(RGB3-Pad1): track 0.00 -> 56.0 mm
- net COL7: track 113.2 -> 168.7 mm
- net Net-(RGB7-Pad1): track 0.00 -> 47.3 mm
- net Net-(RGB10-Pad3): track 0.00 -> 46.7 mm
- net ROW8: track 267.7 -> 312.3 mm
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
Commit message: Finished traces and added ground fills
Parts:
- moved D79 34.9 mm to (242.9, -212.7)
- moved R87 33.4 mm to (242.9, -200.0)
- moved D72 7.32 mm to (236.5, -212.7)
- moved D77 7.32 mm to (239.7, -212.7)
- moved R82 1.59 mm to (236.5, -200.0)
- moved R89 1.59 mm to (239.7, -200.0)
Connections:
- J1 pad 1: MISO -> ROW0
- J1 pad 3: SCK -> LEDIND2
- J1 pad 4: MOSI -> LEDIND1
- U1 pad 1: Net-(U1-Pad1) -> ROW1
- U1 pad 10: Net-(U1-Pad10) -> LEDIND1
- U1 pad 11: Net-(U1-Pad11) -> ROW0
- U1 pad 18: Net-(U1-Pad18) -> RGBLED
- U1 pad 19: Net-(U1-Pad19) -> ROW10
- U1 pad 20: Net-(U1-Pad20) -> ROW11
- U1 pad 21: Net-(U1-Pad21) -> ROW9
- U1 pad 22: Net-(U1-Pad22) -> ROW8
- U1 pad 25: Net-(U1-Pad25) -> COL7
- U1 pad 26: Net-(U1-Pad26) -> COL6
- U1 pad 27: Net-(U1-Pad27) -> COL5
- U1 pad 28: Net-(U1-Pad28) -> COL4
- U1 pad 29: Net-(U1-Pad29) -> COL3
- U1 pad 30: Net-(U1-Pad30) -> COL2
- U1 pad 31: Net-(U1-Pad31) -> COL1
- U1 pad 32: Net-(U1-Pad32) -> COL0
- U1 pad 36: Net-(U1-Pad36) -> ROW6
- U1 pad 37: Net-(U1-Pad37) -> ROW7
- U1 pad 38: Net-(U1-Pad38) -> ROW5
- U1 pad 39: Net-(U1-Pad39) -> ROW4
- U1 pad 40: Net-(U1-Pad40) -> ROW2
- U1 pad 41: Net-(U1-Pad41) -> ROW3
- U1 pad 8: Net-(U1-Pad8) -> LEDIND3
- U1 pad 9: Net-(U1-Pad9) -> LEDIND2
Routing:
- net GND: track 217.6 -> 1163.4 mm, vias 2 -> 21
- net +5V: track 2019.3 -> 2577.1 mm, vias 8 -> 15
- net COL0: track 220.9 -> 521.1 mm, vias 0 -> 2
- net COL1: track 229.7 -> 472.7 mm, vias 0 -> 2
- net COL2: track 201.6 -> 407.6 mm, vias 0 -> 2
- net LEDGND: track 1605.0 -> 1792.8 mm, vias 7 -> 17
- net COL3: track 220.7 -> 390.2 mm, vias 0 -> 2
- net COL4: track 235.7 -> 368.6 mm, vias 0 -> 2
- net ROW2: track 219.5 -> 335.3 mm, vias 0 -> 4
- net COL5: track 240.6 -> 337.0 mm, vias 0 -> 2
- net RESET: track 12.1 -> 102.6 mm, vias 2 -> 6
- net ROW6: track 206.0 -> 284.5 mm, vias 0 -> 3
- net ROW3: track 242.3 -> 311.3 mm, vias 0 -> 4
- net COL6: track 217.4 -> 284.2 mm, vias 0 -> 1
- net COL7: track 168.7 -> 233.0 mm, vias 0 -> 2
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- added copper zone on B.Cu, net GND
- added copper zone on F.Cu, net GND

Commit message: Adjusted silkscreen and added edge rails
Parts:
- added Tab1: BreakawayTabs, random-keyboard-parts:breakaway-mousebites, F.Cu at (1.59, -234.2)
- added Tab10: BreakawayTabs, random-keyboard-parts:breakaway-mousebites, F.Cu at (161.1, -119.9)
- added Tab11: BreakawayTabs, random-keyboard-parts:breakaway-mousebites, F.Cu at (122.2, -119.9)
- added Tab12: BreakawayTabs, random-keyboard-parts:breakaway-mousebites, F.Cu at (89.7, -119.9)
- added Tab13: BreakawayTabs, random-keyboard-parts:breakaway-mousebites, F.Cu at (3.97, -119.9)
- added Tab2: BreakawayTabs, random-keyboard-parts:breakaway-mousebites, F.Cu at (44.5, -234.2)
- added Tab3: BreakawayTabs, random-keyboard-parts:breakaway-mousebites, F.Cu at (125.4, -234.2)
- added Tab4: BreakawayTabs, random-keyboard-parts:breakaway-mousebites, F.Cu at (225.4, -234.2)
- added Tab5: BreakawayTabs, random-keyboard-parts:breakaway-mousebites, F.Cu at (267.5, -234.2)
- added Tab6: BreakawayTabs, random-keyboard-parts:breakaway-mousebites, F.Cu at (298.4, -234.2)
- added Tab7: BreakawayTabs, random-keyboard-parts:breakaway-mousebites, F.Cu at (292.9, -115.9)
- added Tab8: BreakawayTabs, random-keyboard-parts:breakaway-mousebites, F.Cu at (254.8, -115.9)
- added Tab9: BreakawayTabs, random-keyboard-parts:breakaway-mousebites, F.Cu at (225.4, -119.9)
- moved D76 0.79 mm to (276.2, -223.8)
- moved D83 0.79 mm to (290.5, -223.8)
Routing:
- net ROW0: track 339.9 -> 337.8 mm
Other:
- board size 315.1 x 125.4 mm -> 315.1 x 150.8 mm
