File: Asok75.sch (KiCad schematic (older format))
At the start: 349 parts, among them J1 AVR-ISP-6, Q1 2N7002, SW1 SW_Push, U1 ATmega32U4-MU, U2 PRTR5V0U2X, Y1 16MHz

Commit message: Removed extra symbols in schematic in hotswap variant
Parts:
- C1, C10, C11, C12, C13, C14, C15, C16, C17, C18, C19, C2, C20, C21, C3, C4, C5, C6, C7, C8, C9: footprint Capacitor_SMD:C_0805_2012Metric -> Capacitor_SMD:C_0603_1608Metric
- R1, R10, R11, R12, R13, R14, R15, R16, R17, R18, R19, R2, R20, R21, R22, R23, R24, R25, R26, R27, R28, R29, R3, R30, R31, R32, R33, R34, R35, R36, R37, R38, R39, R4, R40, R41, R42, R43, R44, R45, R46, R47, R48, R49, R5, R50, R51, R52, R53, R54, R55, R56, R57, R58, R59, R6, R60, R61, R62, R63, R64, R65, R66, R67, R68, R69, R7, R70, R71, R72, R73, R74, R75, R76, R77, R78, R79, R8, R80, R81, R82, R83, R84, R85, R86, R87, R88, R89, R9, R90, R91, R92, R93, R94, R95, R96, R97, R98: footprint Resistor_SMD:R_0805_2012Metric -> Resistor_SMD:R_0603_1608Metric

Commit message: Refactored project into separate repositories
Parts:
- removed LED1, LED10, LED11, LED12, LED13, LED14, LED2, LED3, LED4, LED5, LED6, LED7, LED8, LED9: SK6812-SIDEA-4020, asok75:SK6812-SIDEA-4020, symbol asok75:SK6812-SIDEA-4020
- removed U1: ATmega32U4-MU, Package_DFN_QFN:QFN-44-1EP_7x7mm_P0.5mm_EP5.2x5.2mm, symbol MCU_Microchip_ATmega:ATmega32U4-MU
- added RGB1, RGB10, RGB11, RGB12, RGB13, RGB14, RGB2, RGB3, RGB4, RGB5, RGB6, RGB7, RGB8, RGB9: SK6812MINI, LED_SMD:LED_SK6812MINI_PLCC4_3.5x3.5mm_P1.75mm, symbol LED:SK6812MINI
- added U1: ATmega32U4-AU, Package_QFP:TQFP-44_10x10mm_P0.8mm, symbol MCU_Microchip_ATmega:ATmega32U4-AU
- C1, C10, C11, C12, C13, C14, C15, C16, C17, C18, C19, C2, C20, C21, C3, C4, C5, C6, C7, C8, C9: footprint Capacitor_SMD:C_0603_1608Metric -> Capacitor_SMD:C_0805_2012Metric
- R1, R10, R11, R12, R13, R14, R15, R16, R17, R18, R19, R2, R20, R21, R22, R23, R24, R25, R26, R27, R28, R29, R3, R30, R31, R32, R33, R34, R35, R36, R37, R38, R39, R4, R40, R41, R42, R43, R44, R45, R46, R47, R48, R49, R5, R50, R51, R52, R53, R54, R55, R56, R57, R58, R59, R6, R60, R61, R62, R63, R64, R65, R66, R67, R68, R69, R7, R70, R71, R72, R73, R74, R75, R76, R77, R78, R79, R8, R80, R81, R82, R83, R84, R85, R86, R87, R88, R89, R9, R90, R91, R92, R93, R94, R95, R96, R97, R98: footprint Resistor_SMD:R_0603_1608Metric -> Resistor_SMD:R_0805_2012Metric
Connections:
- net +5V: now also RGB1.4 (VDD), RGB10.4 (VDD), RGB11.4 (VDD), RGB12.4 (VDD), RGB13.4 (VDD), RGB14.4 (VDD), RGB2.4 (VDD), RGB3.4 (VDD), RGB4.4 (VDD), RGB5.4 (VDD), RGB6.4 (VDD), RGB7.4 (VDD), RGB8.4 (VDD), RGB9.4 (VDD), U1.14 (VCC), U1.2 (UVCC), U1.24 (AVCC), U1.34 (VCC), U1.44 (AVCC), U1.7 (VBUS)
- net COL0: now also U1.32 (PC7)
- net COL1: now also U1.31 (PC6)
- net COL2: now also U1.30 (PB6)
- net COL3: now also U1.29 (PB5)
- net COL4: now also U1.28 (PB4)
- net COL5: now also U1.27 (PD7)
- net COL6: now also U1.26 (PD6)
- net COL7: now also U1.25 (PD4)
- net D+: now also U1.4 (D+)
- net D-: now also U1.3 (D-)
- net GND: now also RGB1.2 (VSS), RGB10.2 (VSS), RGB11.2 (VSS), RGB12.2 (VSS), RGB13.2 (VSS), RGB14.2 (VSS), RGB2.2 (VSS), RGB3.2 (VSS), RGB4.2 (VSS), RGB5.2 (VSS), RGB6.2 (VSS), RGB7.2 (VSS), RGB8.2 (VSS), RGB9.2 (VSS), U1.15 (GND), U1.23 (GND), U1.35 (GND), U1.43 (GND), U1.5 (UGND)
- net LEDIND1: now also U1.10 (PB2)
- net LEDIND2: now also U1.9 (PB1)
- net LEDIND3: now also U1.8 (PB0)
- net LEDMOS: now also U1.12 (PB7)
- net RESET: now also U1.13 (~RESET)
- net RGBLED: now also RGB1.3 (DIN), U1.18 (PD0)
- net ROW0: now also U1.1 (PE6)
- net ROW1: now also U1.11 (PB3)
- net ROW10: now also U1.20 (PD2)
- net ROW11: now also U1.19 (PD1)
- net ROW2: now also U1.41 (PF0)
- net ROW3: now also U1.40 (PF1)
- net ROW4: now also U1.39 (PF4)
- net ROW5: now also U1.38 (PF5)
- net ROW6: now also U1.37 (PF6)
- net ROW7: now also U1.36 (PF7)
- net ROW8: now also U1.21 (PD3)
- net ROW9: now also U1.22 (PD5)
- net at R4.2: now also U1.33 (~HWB~/PE2)
- net at C1.1, Y1.1: now also U1.17 (XTAL1)
- net at C2.1, Y1.3: now also U1.16 (XTAL2)
- net at C7.1: now also U1.6 (UCAP)
- new net: RGB1.1 (DOUT), RGB2.3 (DIN)
- new net: RGB2.1 (DOUT), RGB3.3 (DIN)
- new net: RGB3.1 (DOUT), RGB4.3 (DIN)
- new net: RGB4.1 (DOUT), RGB5.3 (DIN)
- new net: RGB8.1 (DOUT), RGB9.3 (DIN)
- new net: RGB7.1 (DOUT), RGB8.3 (DIN)
- new net: RGB10.3 (DIN), RGB9.1 (DOUT)
- new net: RGB10.1 (DOUT), RGB11.3 (DIN)
- new net: RGB11.1 (DOUT), RGB12.3 (DIN)
- new net: RGB5.1 (DOUT), RGB6.3 (DIN)
- new net: RGB6.1 (DOUT), RGB7.3 (DIN)
- new net: RGB12.1 (DOUT), RGB13.3 (DIN)
- new net: RGB13.1 (DOUT), RGB14.3 (DIN)

Commit message: Deleted traces, updated dimensions, added new symbols and footprints for side firing underglow LEDS
Parts:
- removed RGB1, RGB10, RGB11, RGB12, RGB13, RGB14, RGB2, RGB3, RGB4, RGB5, RGB6, RGB7, RGB8, RGB9: SK6812MINI, LED_SMD:LED_SK6812MINI_PLCC4_3.5x3.5mm_P1.75mm, symbol LED:SK6812MINI
- removed U1: ATmega32U4-AU, Package_QFP:TQFP-44_10x10mm_P0.8mm, symbol MCU_Microchip_ATmega:ATmega32U4-AU
- added LED1, LED10, LED11, LED12, LED13, LED14, LED2, LED3, LED4, LED5, LED6, LED7, LED8, LED9: SK6812-SIDEA-4020, asok75:SK6812-SIDEA-4020, symbol asok75:SK6812-SIDEA-4020
- added U1: ATmega32U4-MU, Package_DFN_QFN:QFN-44-1EP_7x7mm_P0.5mm_EP5.2x5.2mm, symbol MCU_Microchip_ATmega:ATmega32U4-MU
Connections:
- net +5V: now also LED1.2 (VCC), LED10.2 (VCC), LED11.2 (VCC), LED12.2 (VCC), LED13.2 (VCC), LED14.2 (VCC), LED2.2 (VCC), LED3.2 (VCC), LED4.2 (VCC), LED5.2 (VCC), LED6.2 (VCC), LED7.2 (VCC), LED8.2 (VCC), LED9.2 (VCC), U1.14 (VCC), U1.2 (UVCC), U1.24 (AVCC), U1.34 (VCC), U1.44 (AVCC), U1.7 (VBUS)
- net COL0: now also U1.32 (PC7)
- net COL1: now also U1.31 (PC6)
- net COL2: now also U1.30 (PB6)
- net COL3: now also U1.29 (PB5)
- net COL4: now also U1.28 (PB4)
- net COL5: now also U1.27 (PD7)
- net COL6: now also U1.26 (PD6)
- net COL7: now also U1.25 (PD4)
- net D+: now also U1.4 (D+)
- net D-: now also U1.3 (D-)
- net GND: now also LED1.4 (GND), LED10.4 (GND), LED11.4 (GND), LED12.4 (GND), LED13.4 (GND), LED14.4 (GND), LED2.4 (GND), LED3.4 (GND), LED4.4 (GND), LED5.4 (GND), LED6.4 (GND), LED7.4 (GND), LED8.4 (GND), LED9.4 (GND), U1.15 (GND), U1.23 (GND), U1.35 (GND), U1.43 (GND), U1.45 (GND), U1.5 (UGND)
- net LEDIND1: now also U1.10 (PB2)
- net LEDIND2: now also U1.9 (PB1)
- net LEDIND3: now also U1.8 (PB0)
- net LEDMOS: now also U1.12 (PB7)
- net RESET: now also U1.13 (~RESET)
- net RGBLED: now also LED1.1 (DIN), U1.18 (PD0)
- net ROW0: now also U1.1 (PE6)
- net ROW1: now also U1.11 (PB3)
- net ROW10: now also U1.20 (PD2)
- net ROW11: now also U1.19 (PD1)
- net ROW2: now also U1.41 (PF0)
- net ROW3: now also U1.40 (PF1)
- net ROW4: now also U1.39 (PF4)
- net ROW5: now also U1.38 (PF5)
- net ROW6: now also U1.37 (PF6)
- net ROW7: now also U1.36 (PF7)
- net ROW8: now also U1.21 (PD3)
- net ROW9: now also U1.22 (PD5)
- net at R4.2: now also U1.33 (~HWB~/PE2)
- net at C2.1, Y1.3: now also U1.16 (XTAL2)
- net at C1.1, Y1.1: now also U1.17 (XTAL1)
- net at C7.1: now also U1.6 (UCAP)
- new net: LED1.3 (DOUT), LED2.1 (DIN)
- new net: LED2.3 (DOUT), LED3.1 (DIN)
- new net: LED3.3 (DOUT), LED4.1 (DIN)
- new net: LED4.3 (DOUT), LED5.1 (DIN)
- new net: LED5.3 (DOUT), LED6.1 (DIN)
- new net: LED6.3 (DOUT), LED7.1 (DIN)
- new net: LED7.3 (DOUT), LED8.1 (DIN)
- new net: LED8.3 (DOUT), LED9.1 (DIN)
- new net: LED10.1 (DIN), LED9.3 (DOUT)
- new net: LED10.3 (DOUT), LED11.1 (DIN)
- new net: LED11.3 (DOUT), LED12.1 (DIN)
- new net: LED12.3 (DOUT), LED13.1 (DIN)
- new net: LED13.3 (DOUT), LED14.1 (DIN)
