File: v1.kicad_pcb (KiCad board)
At the start: 2 copper layers, 315.5 x 124.9 mm, 363 parts, among them J1 AVR-ISP-6, Q1 2N7002, SW1 SW_Push, U1 ATmega32U4-MU, U2 PRTR5V0U2X, Y1 16MHz

Commit message: Deleted traces, updated dimensions, added new symbols and footprints for side firing underglow LEDS
Parts:
- removed LED1, LED10, LED11, LED12, LED13, LED14, LED2, LED3, LED4, LED5, LED6, LED7, LED8, LED9: SK6812-SIDEA-4020, asok75:SK6812-SIDEA-4020
- added G***: LOGO, silkscreen:southerncross-mask, B.Cu at (262.7, -138.1)
- added G***: LOGO, silkscreen:southerncross, B.Cu at (262.7, -138.1)
- U1: value ATmega32U4-MU -> ATmega32U4-AU; footprint Package_DFN_QFN:QFN-44-1EP_7x7mm_P0.5mm_EP5.2x5.2mm -> Package_QFP:TQFP-44_10x10mm_P0.8mm
- moved Tab1 430.9 mm to (1.59, -234.2)
- moved Tab2 402.3 mm to (44.5, -234.2)
- moved Tab3 363.4 mm to (125.4, -234.2)
- moved Tab13 362.0 mm to (3.97, -119.9), turned to 180 degrees
- moved Tab4 331.4 mm to (225.4, -234.2)
- moved Tab5 318.4 mm to (267.5, -234.2)
- moved Tab6 315.4 mm to (298.4, -234.2)
- moved Tab12 294.4 mm to (89.7, -119.9), turned to 180 degrees
- moved USB1 276.9 mm to (283.4, -241.3)
- moved MX_DEL1 276.5 mm to (298.4, -224.6)
- moved MX_END1 276.5 mm to (298.4, -148.4)
- moved MX_HOME1 276.5 mm to (298.4, -205.6)
- moved MX_PGUP1 276.5 mm to (298.4, -186.5)
- moved MX_PGDN1 276.5 mm to (298.4, -167.5)
- moved J1 276.4 mm to (283.4, -197.6)
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Routing:
- net +5V: track 0.00 -> 2574.2 mm, vias 0 -> 16
- net LEDGND: track 0.00 -> 1768.7 mm, vias 0 -> 20
- net GND: track 0.00 -> 1157.2 mm, vias 0 -> 20
- net COL0: track 0.00 -> 520.5 mm, vias 0 -> 2
- net COL1: track 0.00 -> 472.7 mm, vias 0 -> 2
- net COL2: track 0.00 -> 407.6 mm, vias 0 -> 2
- net COL3: track 0.00 -> 390.2 mm, vias 0 -> 2
- net COL4: track 0.00 -> 368.6 mm, vias 0 -> 2
- net ROW8: track 0.00 -> 343.6 mm, vias 0 -> 4
- net COL5: track 0.00 -> 337.0 mm, vias 0 -> 2
- net ROW3: track 0.00 -> 334.8 mm, vias 0 -> 4
- net ROW10: track 0.00 -> 327.3 mm, vias 0 -> 4
- net ROW0: track 0.00 -> 315.5 mm, vias 0 -> 4
- net ROW2: track 0.00 -> 310.1 mm, vias 0 -> 4
- net ROW1: track 0.00 -> 308.5 mm, vias 0 -> 3
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- added copper zone on B.Cu, net GND
- added copper zone on F.Cu, net GND
Other:
- board size 315.5 x 124.9 mm -> 315.1 x 150.8 mm
