File: Asok75.kicad_pcb (KiCad board)
At the start: 2 copper layers, 315.5 x 124.9 mm, 363 parts, among them J1 AVR-ISP-6, Q1 2N7002, SW1 SW_Push, U1 ATmega32U4-MU, U2 PRTR5V0U2X, Y1 16MHz

Commit message: Removed extra symbols in schematic in hotswap variant
Parts:
- removed RGB1, RGB10, RGB11, RGB12, RGB13, RGB14, RGB2, RGB3, RGB4, RGB5, RGB6, RGB7, RGB8, RGB9: SK6812MINI, LED_SMD:LED_SK6812MINI_PLCC4_3.5x3.5mm_P1.75mm
- C1, C10, C11, C12, C13, C14, C15, C16, C17, C18, C19, C2, C20, C21, C3, C4, C5, C6, C7, C8, C9: footprint Capacitor_SMD:C_0805_2012Metric -> Capacitor_SMD:C_0603_1608Metric
- R1, R10, R11, R12, R13, R14, R15, R16, R17, R18, R19, R2, R20, R21, R22, R23, R24, R25, R26, R27, R28, R29, R3, R30, R31, R32, R33, R34, R35, R36, R37, R38, R39, R4, R40, R41, R42, R43, R44, R45, R46, R47, R48, R49, R5, R50, R51, R52, R53, R54, R55, R56, R57, R58, R59, R6, R60, R61, R62, R63, R64, R65, R66, R67, R68, R69, R7, R70, R71, R72, R73, R74, R75, R76, R77, R78, R79, R8, R80, R81, R82, R83, R84, R85, R86, R87, R88, R89, R9, R90, R91, R92, R93, R94, R95, R96, R97, R98: footprint Resistor_SMD:R_0805_2012Metric -> Resistor_SMD:R_0603_1608Metric
- moved R16 403.3 mm to (325.2, -25.7), turned to 0 degrees
- moved R17 394.3 mm to (329.6, -22.8), turned to 0 degrees
- moved R22 376.1 mm to (334.0, -22.8), turned to 0 degrees
- moved R14 375.3 mm to (329.6, -19.8), turned to 0 degrees
- moved R15 373.9 mm to (320.8, -30.3), turned to 0 degrees
- moved R23 372.1 mm to (325.2, -31.6), turned to 0 degrees
- moved R20 371.2 mm to (347.2, -25.7), turned to 0 degrees
- moved R13 371.1 mm to (325.2, -22.8), turned to 0 degrees
- moved R12 363.8 mm to (320.8, -27.3), turned to 0 degrees
- moved R29 362.8 mm to (338.4, -22.8), turned to 0 degrees
- moved R21 356.9 mm to (329.6, -25.7), turned to 0 degrees
- moved R28 356.1 mm to (325.2, -34.6), turned to 0 degrees
- moved R19 354.4 mm to (325.2, -28.7), turned to 0 degrees
- moved R18 351.4 mm to (334.0, -19.8), turned to 0 degrees
- moved R34 346.8 mm to (338.4, -25.7), turned to 0 degrees
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Other:
- board text removed: "Designed by Asok"

Commit message: Updated edge cuts
Parts:
- removed LED1, LED10, LED11, LED12, LED13, LED14, LED2, LED3, LED4, LED5, LED6, LED7, LED8, LED9: SK6812-SIDEA-4020, asok75:SK6812-SIDEA-4020
Other:
- board size 315.5 x 124.9 mm -> 321.9 x 124.1 mm

Commit message: Realigned underglow LEDs
Parts:
- added LED1: SK6812-SIDEA-4020, asok75:SK6812-SIDEA-4020, B.Cu at (263.1, 113.9)
- added LED10: SK6812-SIDEA-4020, asok75:SK6812-SIDEA-4020, B.Cu at (-28.9, 150.5)
- added LED11: SK6812-SIDEA-4020, asok75:SK6812-SIDEA-4020, B.Cu at (64.5, 150.8)
- added LED12: SK6812-SIDEA-4020, asok75:SK6812-SIDEA-4020, B.Cu at (134.8, 151.0)
- added LED13: SK6812-SIDEA-4020, asok75:SK6812-SIDEA-4020, B.Cu at (175.4, 151.0)
- added LED14: SK6812-SIDEA-4020, asok75:SK6812-SIDEA-4020, B.Cu at (241.3, 154.0)
- added LED2: SK6812-SIDEA-4020, asok75:SK6812-SIDEA-4020, B.Cu at (263.1, 75.9)
- added LED3: SK6812-SIDEA-4020, asok75:SK6812-SIDEA-4020, B.Cu at (218.5, 40.8)
- added LED4: SK6812-SIDEA-4020, asok75:SK6812-SIDEA-4020, B.Cu at (159.7, 40.8)
- added LED5: SK6812-SIDEA-4020, asok75:SK6812-SIDEA-4020, B.Cu at (90.2, 41.1)
- added LED6: SK6812-SIDEA-4020, asok75:SK6812-SIDEA-4020, B.Cu at (30.0, 41.2)
- added LED7: SK6812-SIDEA-4020, asok75:SK6812-SIDEA-4020, B.Cu at (-31.9, 41.3)
- added LED8: SK6812-SIDEA-4020, asok75:SK6812-SIDEA-4020, B.Cu at (-49.4, 77.7)
- added LED9: SK6812-SIDEA-4020, asok75:SK6812-SIDEA-4020, B.Cu at (-49.7, 115.7)
- moved R6 0.38 mm to (244.8, 43.1)
- moved U2 0.22 mm to (240.3, 43.7)

Commit message: Updated hotswap PCB
Parts:
- moved LED14 1.63 mm to (241.3, 155.6)
- moved LED10 0.79 mm to (-28.9, 151.3)
- moved LED7 0.50 mm to (-31.9, 40.8)
- moved LED11 0.49 mm to (64.5, 151.3)
- moved LED9 0.45 mm to (-49.2, 115.7)
- moved LED6 0.37 mm to (30.0, 40.8)
- moved LED5 0.30 mm to (90.2, 40.8)
- moved LED12 0.29 mm to (134.8, 151.3)
- moved LED13 0.29 mm to (175.4, 151.3)
- moved LED8 0.22 mm to (-49.2, 77.7)

Commit message: Refactored project into separate repositories
Parts:
- removed LED1, LED10, LED11, LED12, LED13, LED14, LED2, LED3, LED4, LED5, LED6, LED7, LED8, LED9: SK6812-SIDEA-4020, asok75:SK6812-SIDEA-4020
- added G***: LOGO, silkscreen:southerncross-mask, B.Cu at (262.7, -138.1)
- added G***: LOGO, silkscreen:southerncross, B.Cu at (262.7, -138.1)
- added RGB1: SK6812MINI, LED_SMD:LED_SK6812MINI_PLCC4_3.5x3.5mm_P1.75mm, B.Cu at (304.8, -158.8)
- added RGB10: SK6812MINI, LED_SMD:LED_SK6812MINI_PLCC4_3.5x3.5mm_P1.75mm, B.Cu at (13.5, -122.2)
- added RGB11: SK6812MINI, LED_SMD:LED_SK6812MINI_PLCC4_3.5x3.5mm_P1.75mm, B.Cu at (107.2, -122.2)
- added RGB12: SK6812MINI, LED_SMD:LED_SK6812MINI_PLCC4_3.5x3.5mm_P1.75mm, B.Cu at (177.8, -122.2)
- added RGB13: SK6812MINI, LED_SMD:LED_SK6812MINI_PLCC4_3.5x3.5mm_P1.75mm, B.Cu at (218.3, -122.2)
- added RGB14: SK6812MINI, LED_SMD:LED_SK6812MINI_PLCC4_3.5x3.5mm_P1.75mm, B.Cu at (284.2, -118.3)
- added RGB2: SK6812MINI, LED_SMD:LED_SK6812MINI_PLCC4_3.5x3.5mm_P1.75mm, B.Cu at (304.8, -196.8)
- added RGB3: SK6812MINI, LED_SMD:LED_SK6812MINI_PLCC4_3.5x3.5mm_P1.75mm, B.Cu at (261.1, -231.8)
- added RGB4: SK6812MINI, LED_SMD:LED_SK6812MINI_PLCC4_3.5x3.5mm_P1.75mm, B.Cu at (202.4, -231.8)
- added RGB5: SK6812MINI, LED_SMD:LED_SK6812MINI_PLCC4_3.5x3.5mm_P1.75mm, B.Cu at (132.6, -231.8)
- added RGB6: SK6812MINI, LED_SMD:LED_SK6812MINI_PLCC4_3.5x3.5mm_P1.75mm, B.Cu at (73.0, -231.8)
- added RGB7: SK6812MINI, LED_SMD:LED_SK6812MINI_PLCC4_3.5x3.5mm_P1.75mm, B.Cu at (11.1, -231.8)
- added RGB8: SK6812MINI, LED_SMD:LED_SK6812MINI_PLCC4_3.5x3.5mm_P1.75mm, B.Cu at (-5.56, -195.3)
- added RGB9: SK6812MINI, LED_SMD:LED_SK6812MINI_PLCC4_3.5x3.5mm_P1.75mm, B.Cu at (-5.56, -157.2)
- C1, C10, C11, C12, C13, C14, C15, C16, C17, C18, C19, C2, C20, C21, C3, C4, C5, C6, C7, C8, C9: footprint Capacitor_SMD:C_0603_1608Metric -> Capacitor_SMD:C_0805_2012Metric
- R1, R10, R11, R12, R13, R14, R15, R16, R17, R18, R19, R2, R20, R21, R22, R23, R24, R25, R26, R27, R28, R29, R3, R30, R31, R32, R33, R34, R35, R36, R37, R38, R39, R4, R40, R41, R42, R43, R44, R45, R46, R47, R48, R49, R5, R50, R51, R52, R53, R54, R55, R56, R57, R58, R59, R6, R60, R61, R62, R63, R64, R65, R66, R67, R68, R69, R7, R70, R71, R72, R73, R74, R75, R76, R77, R78, R79, R8, R80, R81, R82, R83, R84, R85, R86, R87, R88, R89, R9, R90, R91, R92, R93, R94, R95, R96, R97, R98: footprint Resistor_SMD:R_0603_1608Metric -> Resistor_SMD:R_0805_2012Metric
- U1: value ATmega32U4-MU -> ATmega32U4-AU; footprint Package_DFN_QFN:QFN-44-1EP_7x7mm_P0.5mm_EP5.2x5.2mm -> Package_QFP:TQFP-44_10x10mm_P0.8mm
- moved Tab1 430.9 mm to (1.59, -234.2)
- moved Tab2 402.3 mm to (44.5, -234.2)
- moved R12 364.3 mm to (9.53, -216.7), turned to 90 degrees
- moved Tab3 363.4 mm to (125.4, -234.2)
- moved R13 362.0 mm to (9.53, -200.0), turned to 90 degrees
- moved Tab13 362.0 mm to (3.97, -119.9), turned to 180 degrees
- moved R18 360.7 mm to (33.3, -219.1), turned to 90 degrees
- moved R14 354.1 mm to (14.3, -181.0), turned to 90 degrees
- moved R16 349.4 mm to (-3.97, -142.9), turned to 90 degrees
- moved R24 348.6 mm to (52.4, -219.1), turned to 90 degrees
- moved R20 345.9 mm to (38.1, -181.0), turned to 90 degrees
- moved R19 342.5 mm to (28.6, -200.0), turned to 90 degrees
- moved R17 333.4 mm to (14.3, -131.0), turned to 90 degrees
- moved Tab4 331.4 mm to (225.4, -234.2)
- moved R15 330.6 mm to (17.5, -161.9), turned to 90 degrees
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Routing:
- net +5V: track 0.00 -> 2574.0 mm, vias 0 -> 16
- net LEDGND: track 0.00 -> 1768.7 mm, vias 0 -> 20
- net GND: track 0.00 -> 1157.2 mm, vias 0 -> 20
- net COL0: track 0.00 -> 520.5 mm, vias 0 -> 2
- net COL1: track 0.00 -> 472.7 mm, vias 0 -> 2
- net COL2: track 0.00 -> 407.6 mm, vias 0 -> 2
- net COL3: track 0.00 -> 390.2 mm, vias 0 -> 2
- net COL4: track 0.00 -> 368.6 mm, vias 0 -> 2
- net ROW8: track 0.00 -> 343.6 mm, vias 0 -> 4
- net COL5: track 0.00 -> 337.0 mm, vias 0 -> 2
- net ROW3: track 0.00 -> 334.8 mm, vias 0 -> 4
- net ROW10: track 0.00 -> 327.3 mm, vias 0 -> 4
- net ROW0: track 0.00 -> 315.5 mm, vias 0 -> 4
- net ROW2: track 0.00 -> 310.1 mm, vias 0 -> 4
- net ROW1: track 0.00 -> 308.5 mm, vias 0 -> 3
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- added copper zone on B.Cu, net GND
- added copper zone on F.Cu, net GND
Other:
- board size 321.9 x 124.1 mm -> 315.1 x 150.8 mm
- board text added: "Designed by Asok"
