File: HotSwap/Asok75hotswap2.kicad_pcb (KiCad board)
At the start: 2 copper layers, 314.8 x 124.2 mm, 233 parts, among them J1 AVR-ISP-6, SW1 SW_Push, U1 PRTR5V0U2X, U2 ATmega32U4-MU, Y1 16MHz

Commit message: Updated edge cuts
Parts:
- moved Y1 5.64 mm to (231.9, 86.6), turned to 0 degrees
- moved C16 1.48 mm to (235.4, 86.7)
- turned U2 to 0 degrees
Routing:
- net GND: track 66.5 -> 0.00 mm, vias 2 -> 0
- net COL7: track 58.1 -> 0.00 mm, vias 6 -> 0
- net +5V: track 53.3 -> 0.00 mm, vias 8 -> 0
- net D-: track 49.0 -> 0.00 mm
- net D+: track 48.6 -> 0.00 mm
- net VCC: track 18.8 -> 0.00 mm, vias 1 -> 0
- net Net-(R8-Pad2): track 18.4 -> 0.00 mm, vias 2 -> 0
- net Net-(R7-Pad2): track 17.6 -> 0.00 mm, vias 1 -> 0
- net Net-(C15-Pad1): track 12.4 -> 0.00 mm
- net Net-(C16-Pad1): track 7.64 -> 0.00 mm
- net Net-(C21-Pad1): track 5.51 -> 0.00 mm
- net Net-(R9-Pad2): track 5.39 -> 0.00 mm
- net Net-(R5-Pad2): track 4.92 -> 0.00 mm, vias 1 -> 0
- net Net-(R4-Pad2): track 4.55 -> 0.00 mm, vias 1 -> 0
