File: HotSwap/Asok75hotswap.kicad_pcb (KiCad board)
At the start: 2 copper layers, 315.5 x 124.9 mm, 259 parts, among them J1 AVR-ISP-6, SW1 SW_Push, U1 ATmega32U4-MU, U2 PRTR5V0U2X, Y1 16MHz

Commit message: Removed extra symbols in schematic in hotswap variant
Parts:
- removed the C5 at (244.5, 106.4)
- removed the C7 at (242.9, 85.7)
- removed the D12 at (-9.53, 124.6)
- removed the D30 at (54.8, 143.7)
- removed the D52 at (126.2, 143.7)
- removed the D77 at (196.8, 60.3)
- removed MX_BCKSP2, MX_BCKSP3, MX_LSHIFT3, MX_LWIN2, MX_\2: MX-LED, MX_Only:MXOnly-1U-Hotswap
- removed MX_CAPS2, MX_LSHIFT2, MX_SPACE4: MX-LED, MX_Only:MXOnly-1.25U-Hotswap
- removed MX_ENTER2: MX-LED, MX_Only:MXOnly-ISO-ROTATED-ReversedStabilizers-NoLED
- removed MX_LALT2, MX_LALT3, MX_LCTRL2, MX_RALT2, MX_RCTRL2: MX-LED, MX_Only:MXOnly-1.5U-Hotswap
- removed MX_SPACE2, MX_SPACE3: MX-LED, MX_Only:MXOnly-7U-Hotswap-ReversedStabilizers
- removed MX_SPACE5: MX-LED, MX_Only:MXOnly-2.75U-Hotswap-ReversedStabilizers
- removed MX_SPACE6: MX-LED, MX_Only:MXOnly-2.25U-Hotswap-ReversedStabilizers
- removed the R9 at (239.7, 85.7)
- removed the U1 at (240.5, 96.0)
- added C19: 0.1uF, Capacitor_SMD:C_0603_1608Metric, B.Cu at (244.5, 102.4)
- added C21: 1uF, Capacitor_SMD:C_0603_1608Metric, B.Cu at (241.3, 89.7)
- added R8: 22, Resistor_SMD:R_0603_1608Metric, B.Cu at (239.7, 89.7)
- added U2: ATmega32U4-MU, Package_DFN_QFN:QFN-44-1EP_7x7mm_P0.5mm_EP5.2x5.2mm, B.Cu at (240.3, 96.0)
- C1: renamed from C21; footprint Capacitor_SMD:C_0805_2012Metric -> Capacitor_SMD:C_0603_1608Metric
- C10: renamed from C12; footprint Capacitor_SMD:C_0805_2012Metric -> Capacitor_SMD:C_0603_1608Metric
- C11: footprint Capacitor_SMD:C_0805_2012Metric -> Capacitor_SMD:C_0603_1608Metric
- C12: renamed from C10; footprint Capacitor_SMD:C_0805_2012Metric -> Capacitor_SMD:C_0603_1608Metric
- C13: renamed from C9; footprint Capacitor_SMD:C_0805_2012Metric -> Capacitor_SMD:C_0603_1608Metric
- C14: renamed from C8; footprint Capacitor_SMD:C_0805_2012Metric -> Capacitor_SMD:C_0603_1608Metric
- C15: renamed from C1; footprint Capacitor_SMD:C_0805_2012Metric -> Capacitor_SMD:C_0603_1608Metric
- C16: renamed from C2; footprint Capacitor_SMD:C_0805_2012Metric -> Capacitor_SMD:C_0603_1608Metric
- C17: renamed from C3; footprint Capacitor_SMD:C_0805_2012Metric -> Capacitor_SMD:C_0603_1608Metric
- C18: renamed from C4; footprint Capacitor_SMD:C_0805_2012Metric -> Capacitor_SMD:C_0603_1608Metric
- C2: renamed from C20; footprint Capacitor_SMD:C_0805_2012Metric -> Capacitor_SMD:C_0603_1608Metric
- C20: renamed from C6; footprint Capacitor_SMD:C_0805_2012Metric -> Capacitor_SMD:C_0603_1608Metric
- C3: renamed from C19; footprint Capacitor_SMD:C_0805_2012Metric -> Capacitor_SMD:C_0603_1608Metric
- C4: renamed from C18; footprint Capacitor_SMD:C_0805_2012Metric -> Capacitor_SMD:C_0603_1608Metric
- C5: renamed from C17; footprint Capacitor_SMD:C_0805_2012Metric -> Capacitor_SMD:C_0603_1608Metric
- C6: renamed from C16; footprint Capacitor_SMD:C_0805_2012Metric -> Capacitor_SMD:C_0603_1608Metric
- C7: renamed from C15; footprint Capacitor_SMD:C_0805_2012Metric -> Capacitor_SMD:C_0603_1608Metric
- C8: renamed from C14; footprint Capacitor_SMD:C_0805_2012Metric -> Capacitor_SMD:C_0603_1608Metric
- C9: renamed from C13; footprint Capacitor_SMD:C_0805_2012Metric -> Capacitor_SMD:C_0603_1608Metric
- R1, R2, R3: footprint Resistor_SMD:R_0805_2012Metric -> Resistor_SMD:R_0603_1608Metric
- R4: renamed from R7; footprint Resistor_SMD:R_0805_2012Metric -> Resistor_SMD:R_0603_1608Metric
- R5: renamed from R6; footprint Resistor_SMD:R_0805_2012Metric -> Resistor_SMD:R_0603_1608Metric
- R6: renamed from R5; footprint Resistor_SMD:R_0805_2012Metric -> Resistor_SMD:R_0603_1608Metric
- R7: renamed from R8; footprint Resistor_SMD:R_0805_2012Metric -> Resistor_SMD:R_0603_1608Metric
- R9: renamed from R4; footprint Resistor_SMD:R_0805_2012Metric -> Resistor_SMD:R_0603_1608Metric
- moved D34 16.4 mm to (89.7, 54.8), turned to 180 degrees
- moved D74 16.4 mm to (232.6, 54.8), turned to 180 degrees
- moved SW1 12.7 mm to (240.3, 109.5)
- moved C11 8.29 mm to (154.8, 42.1), turned to 90 degrees
- moved D79 7.94 mm to (247.7, 59.5), turned to 180 degrees
- moved D50 6.40 mm to (151.6, 54.8), turned to 180 degrees
- moved D68 6.40 mm to (208.8, 54.8), turned to 180 degrees
- moved D24 6.40 mm to (46.8, 54.8), turned to 180 degrees
- moved D29 6.40 mm to (70.6, 54.8), turned to 180 degrees
- moved D45 6.40 mm to (127.8, 54.8), turned to 180 degrees
- moved D13 6.40 mm to (8.73, 54.8), turned to 180 degrees
- moved D7 6.40 mm to (-10.3, 54.8), turned to 180 degrees
- moved D40 6.40 mm to (108.7, 54.8), turned to 180 degrees
- moved D56 6.40 mm to (170.7, 54.8), turned to 180 degrees
- moved D62 6.40 mm to (189.7, 54.8), turned to 180 degrees
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- renumbered D2 to D1, D11 to D10, D18 to D11, D13 to D12, D14 to D13, D15 to D14, D16 to D15, D17 to D16, D24 to D17, D19 to D18, D20 to D19, D3 to D2, D21 to D20, D22 to D21, D23 to D22, D29 to D23, D25 to D24, D26 to D25, D27 to D26, D28 to D27, D35 to D28, D31 to D29, D4 to D3, D32 to D30, D33 to D31, D34 to D32, D40 to D33, D36 to D34, D37 to D35, D38 to D36, D39 to D37, D46 to D38, D41 to D39, D5 to D4, D42 to D40, D43 to D41, D44 to D42, D45 to D43, D51 to D44, D47 to D45, D48 to D46, D49 to D47, D50 to D48, D57 to D49, D6 to D5, D53 to D50, D54 to D51, D55 to D52, D56 to D53, D63 to D54, D58 to D55, D59 to D56, D60 to D57, D61 to D58, D62 to D59, D7 to D6, D69 to D60, D64 to D61, D65 to D62, D66 to D63, D67 to D64, D68 to D65, D74 to D66, D70 to D67, D71 to D68, D72 to D69, D8 to D7, D73 to D70, D80 to D71, D81 to D72, D75 to D73, D76 to D74, D79 to D75, D78 to D76, D82 to D77, D83 to D78, D84 to D79, D9 to D8, D85 to D80, D89 to D81, D90 to D82, D91 to D83, D86 to D84, D87 to D85, D88 to D86, D1 to D87, D10 to D9, LED12 to LED10, LED6 to LED11, LED13 to LED12, LED7 to LED13, LED8 to LED2, LED2 to LED3, LED9 to LED4, LED3 to LED5, LED10 to LED6, LED4 to LED7, LED11 to LED8, LED5 to LED9, MX_#0 to MX_#10, U2 to U1
Connections:
- D11 pad 1: ROW8 -> ROW9
- D17 pad 1: ROW9 -> ROW8
- D23 pad 1: ROW8 -> ROW9
- D28 pad 1: ROW9 -> ROW8
- D33 pad 1: ROW8 -> ROW9
- D38 pad 1: ROW9 -> ROW8
- D44 pad 1: ROW8 -> ROW9
- D49 pad 1: ROW9 -> ROW8
- D54 pad 1: ROW8 -> ROW9
- D60 pad 1: ROW9 -> ROW8
- D66 pad 1: ROW8 -> ROW9
- D75 pad 1: ROW2 -> ROW3
- D77 pad 1: ROW10 -> ROW11
- D78 pad 1: ROW1 -> ROW0
- D79 pad 1: ROW3 -> ROW2
- D80 pad 1: ROW5 -> ROW4
- D81 pad 1: ROW7 -> ROW6
- D82 pad 1: ROW9 -> ROW8
- D83 pad 1: ROW11 -> ROW10
- MX_.1 pad 1: COL5 -> COL4
- MX_B1 pad 1: COL3 -> COL2
- MX_BCKSP1 pad 1: COL7 -> COL6
- MX_C1 pad 1: COL2 -> COL1
- MX_DOWN1 pad 1: COL7 -> COL6
- MX_M1 pad 1: COL4 -> COL3
- MX_RSHIFT1 pad 1: COL6 -> COL5
- MX_UP1 pad 1: COL7 -> COL6
- MX_Z1 pad 1: COL1 -> COL0

Commit message: Updated PCB dimensions and component placement on hotswap variant
Parts:
- moved Tab10 131.2 mm to (429.9, 90.6)
- moved Tab11 131.2 mm to (432.3, 85.0)
- moved Tab12 131.2 mm to (432.3, 86.9)
- moved Tab13 131.2 mm to (432.3, 88.8)
- moved Tab2 131.2 mm to (425.5, 83.1)
- moved Tab5 131.2 mm to (425.5, 85.0)
- moved Tab6 131.2 mm to (432.3, 83.1)
- moved Tab7 131.2 mm to (425.5, 86.9)
- moved Tab9 131.2 mm to (425.5, 88.8)
- moved Tab1 131.2 mm to (416.2, 92.4)
- moved Tab3 131.2 mm to (416.2, 94.3)
- moved Tab4 131.2 mm to (423.0, 92.4)
- moved Tab8 131.2 mm to (423.0, 94.3)
- moved D61 43.0 mm to (155.6, 146.8), turned to 0 degrees
- moved D39 24.0 mm to (76.2, 146.8), turned to 0 degrees
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Other:
- board size 315.5 x 124.9 mm -> 314.8 x 124.2 mm

Commit message: Updated underglow LED footprint
Parts:
- removed H1, H2, H3: MountingHole, mounting_hole:mounting
- moved LED2 315.2 mm to (255.0, 73.1), turned to 270 degrees
- moved LED13 236.5 mm to (167.0, 149.0), turned to 180 degrees
- moved LED7 191.6 mm to (-40.5, 37.9)
- moved LED4 191.6 mm to (151.1, 37.9)
- moved LED10 163.5 mm to (-37.3, 149.0)
- moved LED9 158.3 mm to (-57.9, 113.1), turned to 90 degrees
- moved LED8 135.6 mm to (-57.9, 75.1), turned to 90 degrees
- moved LED5 128.6 mm to (81.6, 37.9)
- moved LED6 125.4 mm to (21.4, 37.9), turned to 0 degrees
- moved LED11 116.1 mm to (56.0, 149.0), turned to 180 degrees
- moved LED3 56.8 mm to (210.2, 37.9), turned to 0 degrees
- moved LED12 40.8 mm to (126.3, 149.0)
- moved C15 11.2 mm to (234.2, 88.9), turned to 90 degrees
- moved C17 10.1 mm to (225.6, 96.8)
- moved C16 9.61 mm to (237.3, 85.7), turned to 180 degrees
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Other:
- outline, holes or cut-outs redrawn
- board text removed: "Designed by Asok"

Commit message: Routed USB and MCU area for hotswap version
Parts:
- removed D87: Schottky, random-keyboard-parts:D_SOD-123-Pretty
- moved R8 36.6 mm to (228.6, 48.8)
- moved R7 36.2 mm to (227.0, 48.8)
- moved F1 12.1 mm to (224.6, 45.2)
- moved C15 5.08 mm to (237.3, 84.9), turned to 180 degrees
- moved U1 4.95 mm to (231.9, 41.3)
- moved R4 4.36 mm to (227.0, 40.5)
- moved R5 4.15 mm to (236.5, 40.5)
- moved C16 3.37 mm to (234.9, 88.1), turned to 90 degrees
- moved C19 1.59 mm to (231.9, 103.2), turned to 180 degrees
- moved R9 1.59 mm to (231.9, 104.8)
- moved Y1 0.79 mm to (237.3, 88.1), turned to 270 degrees
- moved LED12 0.52 mm to (126.7, 148.7)
- moved LED7 0.48 mm to (-40.1, 38.2)
- moved LED6 0.48 mm to (21.8, 38.2)
- moved LED4 0.40 mm to (151.4, 38.1)
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Connections:
- F1 pad 1: Net-(D87-Pad2) -> +5V
Routing:
- net GND: track 0.00 -> 66.5 mm, vias 0 -> 2
- net COL7: track 0.00 -> 58.1 mm, vias 0 -> 6
- net +5V: track 0.00 -> 53.3 mm, vias 0 -> 8
- net D-: track 0.00 -> 49.0 mm
- net D+: track 0.00 -> 48.6 mm
- net VCC: track 0.00 -> 18.8 mm, vias 0 -> 1
- net Net-(R8-Pad2): track 0.00 -> 18.4 mm, vias 0 -> 2
- net Net-(R7-Pad2): track 0.00 -> 17.6 mm, vias 0 -> 1
- net Net-(C15-Pad1): track 0.00 -> 12.4 mm
- net Net-(C16-Pad1): track 0.00 -> 7.64 mm
- net Net-(C21-Pad1): track 0.00 -> 5.51 mm
- net Net-(R9-Pad2): track 0.00 -> 5.39 mm
- net Net-(R5-Pad2): track 0.00 -> 4.92 mm, vias 0 -> 1
- net Net-(R4-Pad2): track 0.00 -> 4.55 mm, vias 0 -> 1

Commit message: Updated edge cuts
Parts:
- removed the C19 at (231.9, 103.2)
- removed the C21 at (227.0, 89.7)
- removed the C6 at (-54.8, 113.1)
- removed the D63 at (165.9, 69.8)
- removed the D73 at (209.3, 150.8)
- removed the D79 at (240.9, 69.8)
- removed the D83 at (247.4, 150.8)
- removed the R8 at (228.6, 48.8)
- added C16: 0.1uF, Capacitor_SMD:C_0603_1608Metric, B.Cu at (-45.2, 115.9)
- added C5: 0.1uF, Capacitor_SMD:C_0603_1608Metric, B.Cu at (244.5, 106.4)
- added C7: 1uF, Capacitor_SMD:C_0603_1608Metric, B.Cu at (242.9, 85.7)
- added D1: Schottky, random-keyboard-parts:D_SOD-123-Pretty, B.Cu at (233.4, 54.0)
- added D12: SOD-123, random-keyboard-parts:D_SOD-123-Pretty, B.Cu at (-9.53, 124.6)
- added D30: SOD-123, random-keyboard-parts:D_SOD-123-Pretty, B.Cu at (54.8, 143.7)
- added D52: SOD-123, random-keyboard-parts:D_SOD-123-Pretty, B.Cu at (126.2, 143.7)
- added D66: SOD-123, random-keyboard-parts:D_SOD-123-Pretty, B.Cu at (176.2, 67.5)
- added D75: SOD-123, random-keyboard-parts:D_SOD-123-Pretty, B.Cu at (227.8, 139.7)
- added D82: SOD-123, random-keyboard-parts:D_SOD-123-Pretty, B.Cu at (231.0, 139.7)
- added D84: SOD-123, random-keyboard-parts:D_SOD-123-Pretty, B.Cu at (247.7, 67.5)
- added D91: SOD-123, random-keyboard-parts:D_SOD-123-Pretty, B.Cu at (234.2, 139.7)
- added H1: MountingHole, mounting_hole:mounting, F.Cu at (-24.6, 86.5)
- added H2: MountingHole, mounting_hole:mounting, F.Cu at (77.8, 105.6)
- added H3: MountingHole, mounting_hole:mounting, F.Cu at (208.8, 86.5)
- added MX_BCKSP2: MX-LED, MX_Only:MXOnly-1U, F.Cu at (225.4, 67.5)
- added MX_BCKSP3: MX-LED, MX_Only:MXOnly-1U, F.Cu at (206.4, 67.5)
- added MX_CAPS2: MX-LED, MX_Only:MXOnly-1.25U, F.Cu at (-38.9, 105.6)
- added MX_ENTER2: MX-LED, MX_Only:MXOnly-ISO-ROTATED-ReversedStabilizers, F.Cu at (223.0, 96.0)
- added MX_LALT2: MX-LED, MX_Only:MXOnly-1.5U-FLIPPED, F.Cu at (11.1, 143.7)
- added MX_LALT3: MX-LED, MX_Only:MXOnly-1.5U, F.Cu at (-7.94, 143.7)
- added MX_LCTRL2: MX-LED, MX_Only:MXOnly-1.5U-FLIPPED, F.Cu at (-36.5, 143.7)
- added MX_LSHIFT2: MX-LED, MX_Only:MXOnly-1.25U, F.Cu at (-38.9, 124.6)
- added MX_LSHIFT3: MX-LED, MX_Only:MXOnly-1U, F.Cu at (-17.5, 124.6)
- added MX_LWIN2: MX-LED, MX_Only:MXOnly-1U-FLIPPED, F.Cu at (-12.7, 143.7)
- added MX_RALT2: MX-LED, MX_Only:MXOnly-1.5U, F.Cu at (154.0, 143.7)
- added MX_RCTRL2: MX-LED, MX_Only:MXOnly-1.5U, F.Cu at (182.6, 143.7)
- added MX_SPACE2: MX-LED, MX_Only:MXOnly-7U-ReversedStabilizers, F.Cu at (73.0, 143.7)
- added MX_SPACE3: MX-LED, MX_Only:MXOnly-7U-ReversedStabilizers, F.Cu at (92.1, 143.7)
- added MX_SPACE4: MX-LED, MX_Only:MXOnly-1.25U, F.Cu at (84.9, 143.7)
- added MX_SPACE5: MX-LED, MX_Only:MXOnly-2.75U-ReversedStabilizers, F.Cu at (46.8, 143.7)
- added MX_SPACE6: MX-LED, MX_Only:MXOnly-2.25U-ReversedStabilizers, F.Cu at (118.3, 143.7)
- added MX_\2: MX-LED, MX_Only:MXOnly-1U, F.Cu at (201.6, 105.6)
- added Q1: 2N7002, Package_TO_SOT_SMD:SOT-23, B.Cu at (320.8, -20.6)
- added R10: 100, Resistor_SMD:R_0603_1608Metric, B.Cu at (338.4, -28.7)
- added R11: 10K, Resistor_SMD:R_0603_1608Metric, B.Cu at (320.8, -24.4)
- added R12: 1K, Resistor_SMD:R_0603_1608Metric, B.Cu at (320.8, -27.3)
- added R13: 1K, Resistor_SMD:R_0603_1608Metric, B.Cu at (325.2, -22.8)
- added R14: 1K, Resistor_SMD:R_0603_1608Metric, B.Cu at (329.6, -19.8)
- added R15: 1K, Resistor_SMD:R_0603_1608Metric, B.Cu at (320.8, -30.3)
- added R16: 1K, Resistor_SMD:R_0603_1608Metric, B.Cu at (325.2, -25.7)
- added R17: 1K, Resistor_SMD:R_0603_1608Metric, B.Cu at (329.6, -22.8)
- added R18: 1K, Resistor_SMD:R_0603_1608Metric, B.Cu at (334.0, -19.8)
- added R19: 1K, Resistor_SMD:R_0603_1608Metric, B.Cu at (325.2, -28.7)
- added R20: 1K, Resistor_SMD:R_0603_1608Metric, B.Cu at (347.2, -25.7)
- added R21: 1K, Resistor_SMD:R_0603_1608Metric, B.Cu at (329.6, -25.7)
- added R22: 1K, Resistor_SMD:R_0603_1608Metric, B.Cu at (334.0, -22.8)
- added R23: 1K, Resistor_SMD:R_0603_1608Metric, B.Cu at (325.2, -31.6)
- added R24: 1K, Resistor_SMD:R_0603_1608Metric, B.Cu at (338.4, -19.8)
- added R25: 1K, Resistor_SMD:R_0603_1608Metric, B.Cu at (329.6, -28.7)
- added R26: 1K, Resistor_SMD:R_0603_1608Metric, B.Cu at (320.8, -36.2)
- added R27: 1K, Resistor_SMD:R_0603_1608Metric, B.Cu at (334.0, -25.7)
- added R28: 1K, Resistor_SMD:R_0603_1608Metric, B.Cu at (325.2, -34.6)
- added R29: 1K, Resistor_SMD:R_0603_1608Metric, B.Cu at (338.4, -22.8)
- added R30: 1K, Resistor_SMD:R_0603_1608Metric, B.Cu at (320.8, -39.1)
- added R31: 1K, Resistor_SMD:R_0603_1608Metric, B.Cu at (329.6, -31.6)
- added R32: 1K, Resistor_SMD:R_0603_1608Metric, B.Cu at (320.8, -33.2)
- added R33: 1K, Resistor_SMD:R_0603_1608Metric, B.Cu at (334.0, -28.7)
- added R34: 1K, Resistor_SMD:R_0603_1608Metric, B.Cu at (338.4, -25.7)
- added R35: 1K, Resistor_SMD:R_0603_1608Metric, B.Cu at (320.8, -42.1)
- added R36: 1K, Resistor_SMD:R_0603_1608Metric, B.Cu at (325.2, -37.5)
- added R37: 1K, Resistor_SMD:R_0603_1608Metric, B.Cu at (329.6, -34.6)
- added R38: 1K, Resistor_SMD:R_0603_1608Metric, B.Cu at (342.8, -22.8)
- added R39: 1K, Resistor_SMD:R_0603_1608Metric, B.Cu at (334.0, -31.6)
- added R40: 1K, Resistor_SMD:R_0603_1608Metric, B.Cu at (347.3, -19.8)
- added R41: 1K, Resistor_SMD:R_0603_1608Metric, B.Cu at (325.2, -40.5)
- added R42: 1K, Resistor_SMD:R_0603_1608Metric, B.Cu at (320.8, -45.0)
- added R43: 1K, Resistor_SMD:R_0603_1608Metric, B.Cu at (325.2, -19.8)
- added R44: 1K, Resistor_SMD:R_0603_1608Metric, B.Cu at (342.8, -19.8)
- added R45: 1K, Resistor_SMD:R_0603_1608Metric, B.Cu at (342.8, -25.7)
- added R46: 1K, Resistor_SMD:R_0603_1608Metric, B.Cu at (329.6, -37.5)
- added R47: 1K, Resistor_SMD:R_0603_1608Metric, B.Cu at (334.0, -34.6)
- added R48: 1K, Resistor_SMD:R_0603_1608Metric, B.Cu at (347.3, -22.8)
- added R49: 1K, Resistor_SMD:R_0603_1608Metric, B.Cu at (338.4, -31.6)
- added R50: 1K, Resistor_SMD:R_0603_1608Metric, B.Cu at (325.2, -43.4)
- added R51: 1K, Resistor_SMD:R_0603_1608Metric, B.Cu at (351.7, -19.8)
- added R52: 1K, Resistor_SMD:R_0603_1608Metric, B.Cu at (329.6, -40.5)
- added R53: 1K, Resistor_SMD:R_0603_1608Metric, B.Cu at (342.8, -28.7)
- added R54: 1K, Resistor_SMD:R_0603_1608Metric, B.Cu at (364.9, -19.8)
- added R55: 1K, Resistor_SMD:R_0603_1608Metric, B.Cu at (338.4, -34.6)
- added R56: 1K, Resistor_SMD:R_0603_1608Metric, B.Cu at (351.7, -22.8)
- added R57: 1K, Resistor_SMD:R_0603_1608Metric, B.Cu at (342.8, -31.6)
- added R58: 1K, Resistor_SMD:R_0603_1608Metric, B.Cu at (329.6, -43.4)
- added R59: 1K, Resistor_SMD:R_0603_1608Metric, B.Cu at (356.1, -19.8)
- added R60: 1K, Resistor_SMD:R_0603_1608Metric, B.Cu at (334.0, -40.5)
- added R61: 1K, Resistor_SMD:R_0603_1608Metric, B.Cu at (347.2, -28.7)
- added R62: 1K, Resistor_SMD:R_0603_1608Metric, B.Cu at (351.6, -25.7)
- added R63: 1K, Resistor_SMD:R_0603_1608Metric, B.Cu at (338.4, -37.5)
- added R64: 1K, Resistor_SMD:R_0603_1608Metric, B.Cu at (342.8, -34.6)
- added R65: 1K, Resistor_SMD:R_0603_1608Metric, B.Cu at (364.9, -25.7)
- added R66: 1K, Resistor_SMD:R_0603_1608Metric, B.Cu at (334.0, -37.5)
- added R67: 1K, Resistor_SMD:R_0603_1608Metric, B.Cu at (334.0, -43.4)
- added R68: 1K, Resistor_SMD:R_0603_1608Metric, B.Cu at (360.5, -19.8)
- added R69: 1K, Resistor_SMD:R_0603_1608Metric, B.Cu at (338.4, -40.5)
- added R70: 1K, Resistor_SMD:R_0603_1608Metric, B.Cu at (351.6, -28.7)
- added R71: 1K, Resistor_SMD:R_0603_1608Metric, B.Cu at (356.0, -25.7)
- added R72: 1K, Resistor_SMD:R_0603_1608Metric, B.Cu at (342.8, -37.5)
- added R73: 1K, Resistor_SMD:R_0603_1608Metric, B.Cu at (347.2, -34.6)
- added R74: 1K, Resistor_SMD:R_0603_1608Metric, B.Cu at (360.5, -22.8)
- added R75: 1K, Resistor_SMD:R_0603_1608Metric, B.Cu at (351.6, -31.6)
- added R76: 1K, Resistor_SMD:R_0603_1608Metric, B.Cu at (338.4, -43.4)
- added R77: 1K, Resistor_SMD:R_0603_1608Metric, B.Cu at (356.1, -22.8)
- added R78: 1K, Resistor_SMD:R_0603_1608Metric, B.Cu at (342.8, -40.5)
- added R79: 1K, Resistor_SMD:R_0603_1608Metric, B.Cu at (356.0, -28.7)
- added R80: 1K, Resistor_SMD:R_0603_1608Metric, B.Cu at (360.4, -25.7)
- added R81: 1K, Resistor_SMD:R_0603_1608Metric, B.Cu at (347.2, -37.5)
- added R82: 1K, Resistor_SMD:R_0603_1608Metric, B.Cu at (351.6, -34.6)
- added R83: 1K, Resistor_SMD:R_0603_1608Metric, B.Cu at (364.9, -22.8)
- added R84: 1K, Resistor_SMD:R_0603_1608Metric, B.Cu at (356.0, -31.6)
- added R85: 1K, Resistor_SMD:R_0603_1608Metric, B.Cu at (342.8, -43.4)
- added R86: 1K, Resistor_SMD:R_0603_1608Metric, B.Cu at (347.2, -40.5)
- added R87: 1K, Resistor_SMD:R_0603_1608Metric, B.Cu at (360.4, -28.7)
- added R88: 1K, Resistor_SMD:R_0603_1608Metric, B.Cu at (347.2, -31.6)
- added R89: 1K, Resistor_SMD:R_0603_1608Metric, B.Cu at (351.6, -37.5)
- added R9: 22, Resistor_SMD:R_0603_1608Metric, B.Cu at (239.7, 85.7)
- added R90: 1K, Resistor_SMD:R_0603_1608Metric, B.Cu at (356.0, -34.6)
- added R91: 1K, Resistor_SMD:R_0603_1608Metric, B.Cu at (360.4, -31.6)
- added R92: 1K, Resistor_SMD:R_0603_1608Metric, B.Cu at (347.2, -43.4)
- added R93: 1K, Resistor_SMD:R_0603_1608Metric, B.Cu at (351.6, -40.5)
- added R94: 1K, Resistor_SMD:R_0603_1608Metric, B.Cu at (364.9, -28.7)
- added R95: 1K, Resistor_SMD:R_0603_1608Metric, B.Cu at (356.0, -37.5)
- added R96: 1K, Resistor_SMD:R_0603_1608Metric, B.Cu at (360.4, -34.6)
- added R97: 1K, Resistor_SMD:R_0603_1608Metric, B.Cu at (364.9, -31.6)
- added R98: 1K, Resistor_SMD:R_0603_1608Metric, B.Cu at (351.6, -43.4)
- MX_#0: renamed from MX_#10; footprint MX_Only:MXOnly-1U-Hotswap -> MX_Only:MXOnly-1U
- MX_#1, MX_#2, MX_#3, MX_#4, MX_#5, MX_#6, MX_#7, MX_#8, MX_#9, MX_'1, MX_,1, MX_-1, MX_.1, MX_/1, MX_;1, MX_=1, MX_A1, MX_B1, MX_C1, MX_D1, MX_DEL1, MX_DOWN1, MX_E1, MX_END1, MX_ESC1, MX_F#1, MX_F#10, MX_F#11, MX_F#12, MX_F#2, MX_F#3, MX_F#4, MX_F#5, MX_F#6, MX_F#7, MX_F#8, MX_F#9, MX_F1, MX_G1, MX_H1, MX_HOME1, MX_I1, MX_J1, MX_K1, MX_L1, MX_LEFT1, MX_M1, MX_N1, MX_O1, MX_P1, MX_PAUSE1, MX_PGDN1, MX_PGUP1, MX_Q1, MX_R1, MX_RALT1, MX_RCTRL1, MX_RIGHT1, MX_RWIN1, MX_S1, MX_T1, MX_U1, MX_UP1, MX_V1, MX_W1, MX_X1, MX_Y1, MX_Z1, MX_[1, MX_]1, MX_`1: footprint MX_Only:MXOnly-1U-Hotswap -> MX_Only:MXOnly-1U
- MX_BCKSP1: footprint MX_Only:MXOnly-2U-Hotswap -> MX_Only:MXOnly-2U
- MX_CAPS1, MX_RSHIFT1: footprint MX_Only:MXOnly-1.75U-Hotswap -> MX_Only:MXOnly-1.75U
- MX_ENTER1: footprint MX_Only:MXOnly-2.25U-Hotswap-ReversedStabilizers -> MX_Only:MXOnly-2.25U-ReversedStabilizers
- MX_LALT1, MX_LCTRL1, MX_LWIN1: footprint MX_Only:MXOnly-1.25U-Hotswap -> MX_Only:MXOnly-1.25U
- MX_LSHIFT1: footprint MX_Only:MXOnly-2.25U-Hotswap -> MX_Only:MXOnly-2.25U
- MX_SPACE1: footprint MX_Only:MXOnly-6.25U-Hotswap-ReversedStabilizers -> MX_Only:MXOnly-6.25U-ReversedStabilizers
- MX_TAB1, MX_\1: footprint MX_Only:MXOnly-1.5U-Hotswap -> MX_Only:MXOnly-1.5U
- U1: value PRTR5V0U2X -> ATmega32U4-MU; footprint random-keyboard-parts:SOT143B -> Package_DFN_QFN:QFN-44-1EP_7x7mm_P0.5mm_EP5.2x5.2mm
- U2: value ATmega32U4-MU -> PRTR5V0U2X; footprint Package_DFN_QFN:QFN-44-1EP_7x7mm_P0.5mm_EP5.2x5.2mm -> random-keyboard-parts:SOT143B
- moved C8 308.1 mm to (258.8, 114.3), turned to 90 degrees
- moved C14 291.2 mm to (-31.8, 44.5), turned to 180 degrees
- moved Tab10 131.2 mm to (298.7, 88.8)
- moved Tab11 131.2 mm to (301.1, 83.1)
- moved Tab12 131.2 mm to (301.1, 85.0)
- moved Tab13 131.2 mm to (301.1, 86.9)
- moved Tab2 131.2 mm to (294.2, 81.2)
- moved Tab5 131.2 mm to (294.2, 83.1)
- moved Tab6 131.2 mm to (301.1, 81.2)
- moved Tab7 131.2 mm to (294.2, 85.0)
- moved Tab9 131.2 mm to (294.2, 86.9)
- moved Tab1 131.2 mm to (285.0, 90.5)
- moved Tab3 131.2 mm to (285.0, 92.4)
- moved Tab4 131.2 mm to (291.8, 90.5)
- moved Tab8 131.2 mm to (291.8, 92.4)
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- renumbered C15 to C1, C12 to C10, C10 to C12, C9 to C13, C7 to C15, C5 to C17, C4 to C18, C3 to C19, C16 to C2, C2 to C20, C1 to C21, C17 to C3, C18 to C4, C20 to C6, C13 to C9, D9 to D10, D10 to D11, D12 to D13, D13 to D14, D14 to D15, D15 to D16, D16 to D17, D11 to D18, D18 to D19, D1 to D2, D19 to D20, D20 to D21, D21 to D22, D22 to D23, D17 to D24, D24 to D25, D25 to D26, D26 to D27, D27 to D28, D23 to D29, D2 to D3, D29 to D31, D30 to D32, D31 to D33, D32 to D34, D28 to D35, D34 to D36, D35 to D37, D36 to D38, D37 to D39, D3 to D4, D33 to D40, D39 to D41, D40 to D42, D41 to D43, D42 to D44, D43 to D45, D38 to D46, D45 to D47, D46 to D48, D47 to D49, D4 to D5, D48 to D50, D44 to D51, D50 to D53, D51 to D54, D52 to D55, D53 to D56, D49 to D57, D55 to D58, D56 to D59, D5 to D6, D57 to D60, D58 to D61, D59 to D62, D54 to D63, D61 to D64, D62 to D65, D64 to D67, D65 to D68, D60 to D69, D6 to D7, D67 to D70, D68 to D71, D69 to D72, D70 to D73, D66 to D74, D74 to D76, D76 to D78, D75 to D79, D7 to D8, D71 to D80, D72 to D81, D78 to D83, D80 to D85, D84 to D86, D85 to D87, D86 to D88, D81 to D89, D8 to D9, D82 to D90, R9 to R4, R6 to R5, R5 to R6, R4 to R7, R7 to R8
Connections:
- C1 pad 1: Net-(C15-Pad1) -> Net-(C1-Pad1)
- C2 pad 1: Net-(C16-Pad1) -> Net-(C2-Pad1)
- D18 pad 1: ROW9 -> ROW8
- D24 pad 1: ROW8 -> ROW9
- D29 pad 1: ROW9 -> ROW8
- D35 pad 1: ROW8 -> ROW9
- D40 pad 1: ROW9 -> ROW8
- D46 pad 1: ROW8 -> ROW9
- D51 pad 1: ROW9 -> ROW8
- D57 pad 1: ROW8 -> ROW9
- D63 pad 1: ROW9 -> ROW8
- D69 pad 1: ROW8 -> ROW9
- D74 pad 1: ROW9 -> ROW8
- D77 pad 1: ROW11 -> ROW3
- D79 pad 1: ROW3 -> ROW2
- D83 pad 1: ROW0 -> ROW1
- D85 pad 1: ROW4 -> ROW5
- D89 pad 1: ROW6 -> ROW7
- D90 pad 1: ROW8 -> ROW9
- F1 pad 1: +5V -> Net-(D1-Pad2)
- LED11 pad 1: Net-(LED11-Pad1) -> Net-(LED10-Pad3)
- LED12 pad 1: Net-(LED10-Pad3) -> Net-(LED11-Pad3)
- LED13 pad 1: Net-(LED11-Pad3) -> Net-(LED12-Pad3)
- LED14 pad 1: Net-(LED12-Pad3) -> Net-(LED13-Pad3)
- LED2 pad 1: Net-(LED13-Pad3) -> Net-(LED1-Pad3)
- LED3 pad 1: Net-(LED1-Pad3) -> Net-(LED2-Pad3)
- LED4 pad 1: Net-(LED2-Pad3) -> Net-(LED3-Pad3)
- LED5 pad 1: Net-(LED3-Pad3) -> Net-(LED4-Pad3)
- LED6 pad 1: Net-(LED4-Pad3) -> Net-(LED5-Pad3)
- LED7 pad 1: Net-(LED5-Pad3) -> Net-(LED6-Pad3)
- LED8 pad 1: Net-(LED6-Pad3) -> Net-(LED7-Pad3)
- LED8 pad 3: Net-(LED10-Pad1) -> Net-(LED8-Pad3)
- LED9 pad 1: Net-(LED7-Pad3) -> Net-(LED8-Pad3)
- LED9 pad 3: Net-(LED11-Pad1) -> Net-(LED10-Pad1)
- MX_.1 pad 1: COL4 -> COL5
- MX_B1 pad 1: COL2 -> COL3
- MX_BCKSP1 pad 1: COL6 -> COL7
- MX_C1 pad 1: COL1 -> COL2
- MX_DOWN1 pad 1: COL6 -> COL7
- MX_DOWN1 pad 2: Net-(D77-Pad2) -> Net-(D82-Pad2)
- MX_M1 pad 1: COL3 -> COL4
- MX_RSHIFT1 pad 1: COL5 -> COL6
- MX_UP1 pad 1: COL6 -> COL7
- MX_Z1 pad 1: COL0 -> COL1
- R4 pad 2: Net-(R9-Pad2) -> Net-(R4-Pad2)
- R8 pad 2: Net-(R7-Pad2) (its old number) -> Net-(R8-Pad2)
- U1 pad 1: GND -> ROW0
- U1 pad 2: Net-(R8-Pad2) -> +5V
- U1 pad 3: Net-(R7-Pad2) (its old number) -> D-
- U1 pad 4: VCC -> D+
- U2 pad 1: ROW0 -> GND
- U2 pad 2: +5V -> Net-(R9-Pad2)
- U2 pad 3: D- -> Net-(R8-Pad2)
- U2 pad 4: D+ -> VCC
- USB1 pad 5: Net-(R7-Pad2) (its old number) -> Net-(R8-Pad2)
- USB1 pad 6: Net-(R8-Pad2) -> Net-(R9-Pad2)
- USB1 pad 7: Net-(R7-Pad2) (its old number) -> Net-(R8-Pad2)
- USB1 pad 8: Net-(R8-Pad2) -> Net-(R9-Pad2)
- Y1 pad 1: Net-(C15-Pad1) -> Net-(C1-Pad1)
- Y1 pad 3: Net-(C16-Pad1) -> Net-(C2-Pad1)
Routing:
- net GND: track 66.5 -> 0.00 mm, vias 2 -> 0
- net COL7: track 58.1 -> 0.00 mm, vias 6 -> 0
- net +5V: track 53.3 -> 0.00 mm, vias 8 -> 0
- net D-: track 49.0 -> 0.00 mm
- net D+: track 48.6 -> 0.00 mm
- net VCC: track 18.8 -> 0.00 mm, vias 1 -> 0
- net Net-(R8-Pad2): track 18.4 -> 0.00 mm, vias 2 -> 0
- net Net-(R7-Pad2) (its old number): track 17.6 -> 0.00 mm, vias 1 -> 0
- net Net-(C15-Pad1): track 12.4 -> 0.00 mm
- net Net-(C16-Pad1): track 7.64 -> 0.00 mm
- net Net-(C21-Pad1): track 5.51 -> 0.00 mm
- net Net-(R9-Pad2): track 5.39 -> 0.00 mm
- net Net-(R6-Pad2): track 4.92 -> 0.00 mm, vias 1 -> 0
- net Net-(R7-Pad2): track 4.55 -> 0.00 mm, vias 1 -> 0
Other:
- board size 314.8 x 124.2 mm -> 315.5 x 124.9 mm

Commit message: Updated hotswap PCB
Parts:
- removed the D1 at (233.4, 54.0)
- removed the D12 at (-9.53, 124.6)
- removed the D30 at (54.8, 143.7)
- removed the D52 at (126.2, 143.7)
- removed the D77 at (196.8, 60.3)
- removed H1, H2, H3: MountingHole, mounting_hole:mounting
- removed MX_BCKSP2, MX_BCKSP3, MX_LSHIFT3, MX_\2: MX-LED, MX_Only:MXOnly-1U
- removed MX_CAPS2, MX_LSHIFT2, MX_SPACE4: MX-LED, MX_Only:MXOnly-1.25U
- removed MX_ENTER2: MX-LED, MX_Only:MXOnly-ISO-ROTATED-ReversedStabilizers
- removed MX_LALT2, MX_LCTRL2: MX-LED, MX_Only:MXOnly-1.5U-FLIPPED
- removed MX_LALT3, MX_RALT2, MX_RCTRL2: MX-LED, MX_Only:MXOnly-1.5U
- removed MX_LWIN2: MX-LED, MX_Only:MXOnly-1U-FLIPPED
- removed MX_SPACE2, MX_SPACE3: MX-LED, MX_Only:MXOnly-7U-ReversedStabilizers
- removed MX_SPACE5: MX-LED, MX_Only:MXOnly-2.75U-ReversedStabilizers
- removed MX_SPACE6: MX-LED, MX_Only:MXOnly-2.25U-ReversedStabilizers
- removed Q1: 2N7002, Package_TO_SOT_SMD:SOT-23
- removed R10: 100, Resistor_SMD:R_0603_1608Metric
- removed R11: 10K, Resistor_SMD:R_0603_1608Metric
- removed R12, R13, R14, R15, R16, R17, R18, R19, R20, R21, R22, R23, R24, R25, R26, R27, R28, R29, R30, R31, R32, R33, R34, R35, R36, R37, R38, R39, R40, R41, R42, R43, R44, R45, R46, R47, R48, R49, R50, R51, R52, R53, R54, R55, R56, R57, R58, R59, R60, R61, R62, R63, R64, R65, R66, R67, R68, R69, R70, R71, R72, R73, R74, R75, R76, R77, R78, R79, R80, R81, R82, R83, R84, R85, R86, R87, R88, R89, R90, R91, R92, R93, R94, R95, R96, R97, R98: 1K, Resistor_SMD:R_0603_1608Metric
- MX_#1, MX_#2, MX_#3, MX_#4, MX_#5, MX_#6, MX_#7, MX_#8, MX_#9, MX_'1, MX_,1, MX_-1, MX_.1, MX_/1, MX_;1, MX_=1, MX_A1, MX_B1, MX_C1, MX_D1, MX_DEL1, MX_DOWN1, MX_E1, MX_END1, MX_ESC1, MX_F#1, MX_F#10, MX_F#11, MX_F#12, MX_F#2, MX_F#3, MX_F#4, MX_F#5, MX_F#6, MX_F#7, MX_F#8, MX_F#9, MX_F1, MX_G1, MX_H1, MX_HOME1, MX_I1, MX_J1, MX_K1, MX_L1, MX_LEFT1, MX_M1, MX_N1, MX_O1, MX_P1, MX_PAUSE1, MX_PGDN1, MX_PGUP1, MX_Q1, MX_R1, MX_RALT1, MX_RCTRL1, MX_RIGHT1, MX_RWIN1, MX_S1, MX_T1, MX_U1, MX_UP1, MX_V1, MX_W1, MX_X1, MX_Y1, MX_Z1, MX_[1, MX_]1, MX_`1: footprint MX_Only:MXOnly-1U -> MX_Only:MXOnly-1U-Hotswap
- MX_#10: renamed from MX_#0; footprint MX_Only:MXOnly-1U -> MX_Only:MXOnly-1U-Hotswap
- MX_BCKSP1: footprint MX_Only:MXOnly-2U -> MX_Only:MXOnly-2U-Hotswap
- MX_CAPS1, MX_RSHIFT1: footprint MX_Only:MXOnly-1.75U -> MX_Only:MXOnly-1.75U-Hotswap
- MX_ENTER1: footprint MX_Only:MXOnly-2.25U-ReversedStabilizers -> MX_Only:MXOnly-2.25U-Hotswap-ReversedStabilizers
- MX_LALT1, MX_LCTRL1, MX_LWIN1: footprint MX_Only:MXOnly-1.25U -> MX_Only:MXOnly-1.25U-Hotswap
- MX_LSHIFT1: footprint MX_Only:MXOnly-2.25U -> MX_Only:MXOnly-2.25U-Hotswap
- MX_SPACE1: footprint MX_Only:MXOnly-6.25U-ReversedStabilizers -> MX_Only:MXOnly-6.25U-Hotswap-ReversedStabilizers
- MX_TAB1, MX_\1: footprint MX_Only:MXOnly-1.5U -> MX_Only:MXOnly-1.5U-Hotswap
- moved LED2 311.9 mm to (-49.2, 77.7), turned to 90 degrees
- moved LED13 235.1 mm to (-31.9, 40.8), turned to 0 degrees
- moved LED4 221.8 mm to (-49.2, 115.7), turned to 90 degrees
- moved LED7 211.4 mm to (159.7, 40.8), turned to 0 degrees
- moved LED10 163.7 mm to (134.8, 151.3)
- moved LED5 128.5 mm to (218.5, 40.8)
- moved LED6 125.4 mm to (-28.9, 151.3), turned to 180 degrees
- moved LED9 122.3 mm to (90.2, 40.8)
- moved LED8 118.4 mm to (64.5, 151.3), turned to 180 degrees
- moved LED11 116.0 mm to (30.0, 40.8), turned to 0 degrees
- moved LED3 56.9 mm to (263.1, 75.9), turned to 270 degrees
- moved LED12 40.8 mm to (175.4, 151.3)
- moved C17 38.2 mm to (270.7, 96.8)
- moved R7 37.7 mm to (274.6, 80.2)
- moved R8 29.8 mm to (269.1, 90.5)
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- renumbered C21 to C1, C12 to C10, C10 to C12, C9 to C13, C8 to C14, C1 to C15, C2 to C16, C3 to C17, C4 to C18, C5 to C19, C20 to C2, C6 to C20, C7 to C21, C19 to C3, C18 to C4, C17 to C5, C16 to C6, C15 to C7, C14 to C8, C13 to C9, D2 to D1, D11 to D10, D18 to D11, D13 to D12, D14 to D13, D15 to D14, D16 to D15, D17 to D16, D24 to D17, D19 to D18, D20 to D19, D3 to D2, D21 to D20, D22 to D21, D23 to D22, D29 to D23, D25 to D24, D26 to D25, D27 to D26, D28 to D27, D35 to D28, D31 to D29, D4 to D3, D32 to D30, D33 to D31, D34 to D32, D40 to D33, D36 to D34, D37 to D35, D38 to D36, D39 to D37, D46 to D38, D41 to D39, D5 to D4, D42 to D40, D43 to D41, D44 to D42, D45 to D43, D51 to D44, D47 to D45, D48 to D46, D49 to D47, D50 to D48, D57 to D49, D6 to D5, D53 to D50, D54 to D51, D55 to D52, D56 to D53, D63 to D54, D58 to D55, D59 to D56, D60 to D57, D61 to D58, D62 to D59, D7 to D6, D69 to D60, D64 to D61, D65 to D62, D66 to D63, D67 to D64, D68 to D65, D74 to D66, D70 to D67, D71 to D68, D72 to D69, D8 to D7, D73 to D70, D80 to D71, D81 to D72, D75 to D73, D76 to D74, D79 to D75, D78 to D76, D82 to D77, D83 to D78, D84 to D79, D9 to D8, D85 to D80, D89 to D81, D90 to D82, D91 to D83, D86 to D84, D87 to D85, D88 to D86, D10 to D9, R7 to R4, R6 to R5, R5 to R6, R8 to R7, R9 to R8, R4 to R9, U2 to U1, U1 to U2
Connections:
- D11 pad 1: ROW8 -> ROW9
- D17 pad 1: ROW9 -> ROW8
- D23 pad 1: ROW8 -> ROW9
- D28 pad 1: ROW9 -> ROW8
- D33 pad 1: ROW8 -> ROW9
- D38 pad 1: ROW9 -> ROW8
- D44 pad 1: ROW8 -> ROW9
- D49 pad 1: ROW9 -> ROW8
- D54 pad 1: ROW8 -> ROW9
- D60 pad 1: ROW9 -> ROW8
- D66 pad 1: ROW8 -> ROW9
- D75 pad 1: ROW2 -> ROW3
- D77 pad 1: ROW10 -> ROW11
- D78 pad 1: ROW1 -> ROW0
- D79 pad 1: ROW3 -> ROW2
- D80 pad 1: ROW5 -> ROW4
- D81 pad 1: ROW7 -> ROW6
- D82 pad 1: ROW9 -> ROW8
- D83 pad 1: ROW11 -> ROW10
- F1 pad 1: Net-(D1-Pad2) (its old number) -> +5V
- LED11 pad 1: Net-(LED10-Pad3) -> Net-(LED11-Pad1)
- LED12 pad 1: Net-(LED11-Pad3) -> Net-(LED10-Pad3)
- LED13 pad 1: Net-(LED12-Pad3) -> Net-(LED11-Pad3)
- LED14 pad 1: Net-(LED13-Pad3) -> Net-(LED12-Pad3)
- LED2 pad 1: Net-(LED1-Pad3) -> Net-(LED13-Pad3)
- LED3 pad 1: Net-(LED2-Pad3) -> Net-(LED1-Pad3)
- LED4 pad 1: Net-(LED3-Pad3) -> Net-(LED2-Pad3)
- LED5 pad 1: Net-(LED4-Pad3) -> Net-(LED3-Pad3)
- LED6 pad 1: Net-(LED5-Pad3) -> Net-(LED4-Pad3)
- LED7 pad 1: Net-(LED6-Pad3) -> Net-(LED5-Pad3)
- LED8 pad 1: Net-(LED7-Pad3) -> Net-(LED6-Pad3)
- LED8 pad 3: Net-(LED8-Pad3) -> Net-(LED10-Pad1)
- LED9 pad 1: Net-(LED8-Pad3) -> Net-(LED7-Pad3)
- LED9 pad 3: Net-(LED10-Pad1) -> Net-(LED11-Pad1)
- MX_.1 pad 1: COL5 -> COL4
- MX_B1 pad 1: COL3 -> COL2
- MX_BCKSP1 pad 1: COL7 -> COL6
- MX_C1 pad 1: COL2 -> COL1
- MX_DOWN1 pad 1: COL7 -> COL6
- MX_M1 pad 1: COL4 -> COL3
- MX_RSHIFT1 pad 1: COL6 -> COL5
- MX_UP1 pad 1: COL7 -> COL6
- MX_Z1 pad 1: COL1 -> COL0
Other:
- board size 315.5 x 124.9 mm -> 314.8 x 124.1 mm

Commit message: Completed routing rows, MCU and USB
Parts:
- moved R8 50.2 mm to (237.3, 51.6)
- moved R7 48.3 mm to (235.7, 51.6)
- moved D61 36.8 mm to (161.9, 148.4)
- moved C21 36.8 mm to (233.4, 92.1), turned to 270 degrees
- moved C17 35.7 mm to (234.9, 96.8), turned to 270 degrees
- moved D75 25.2 mm to (222.2, 72.2)
- moved D5 24.3 mm to (-23.0, 129.4)
- moved C16 22.3 mm to (236.2, 83.3), turned to 270 degrees
- moved D76 21.7 mm to (227.0, 91.3)
- moved C19 21.3 mm to (234.9, 87.3)
- moved D6 20.5 mm to (-45.2, 148.4)
- moved C15 18.2 mm to (244.3, 83.3), turned to 90 degrees
- moved D34 15.1 mm to (88.9, 53.2)
- moved D55 15.1 mm to (155.6, 148.4)
- moved D39 14.3 mm to (86.5, 148.4)
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Routing:
- net ROW6: track 0.00 -> 265.5 mm
- net ROW0: track 0.00 -> 258.2 mm
- net ROW4: track 0.00 -> 248.7 mm
- net ROW3: track 0.00 -> 247.8 mm
- net ROW2: track 0.00 -> 243.9 mm
- net ROW5: track 0.00 -> 241.1 mm
- net ROW1: track 0.00 -> 237.9 mm
- net COL5: track 0.00 -> 233.5 mm, vias 0 -> 20
- net ROW7: track 0.00 -> 217.8 mm
- net ROW8: track 0.00 -> 216.6 mm
- net COL6: track 0.00 -> 212.7 mm, vias 0 -> 16
- net ROW9: track 0.00 -> 204.1 mm
- net COL3: track 0.00 -> 113.4 mm, vias 0 -> 10
- net COL0: track 0.00 -> 108.0 mm, vias 0 -> 11
- net +5V: track 0.00 -> 100.8 mm, vias 0 -> 7
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
Commit message: Finished routing columns in hotswap version
Parts:
- moved D83 25.4 mm to (255.3, 153.8)
- moved D73 17.6 mm to (217.2, 153.8)
- moved D77 15.0 mm to (236.3, 153.8)
- moved D80 12.1 mm to (249.6, 91.3)
- moved D78 11.6 mm to (249.6, 53.2)
- moved D79 5.14 mm to (249.6, 72.2)
- moved D82 5.14 mm to (249.6, 129.4)
- moved D81 3.07 mm to (249.6, 110.3)
- moved C5 2.12 mm to (-29.1, 145.5)
- moved D72 1.06 mm to (236.3, 134.7)
- moved D51 0.79 mm to (135.7, 72.2)
- moved D52 0.79 mm to (145.3, 91.3)
- moved D54 0.79 mm to (159.5, 129.4)
- moved D56 0.79 mm to (169.1, 53.2)
- moved D59 0.79 mm to (169.1, 110.3)
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Routing:
- net ROW10: track 0.50 -> 311.3 mm, vias 0 -> 9
- net ROW11: track 0.00 -> 258.8 mm, vias 0 -> 4
- net COL0: track 108.0 -> 226.8 mm, vias 11 -> 20
- net COL1: track 88.3 -> 200.4 mm, vias 8 -> 18
- net COL4: track 94.2 -> 203.4 mm, vias 8 -> 18
- net COL7: track 0.00 -> 103.2 mm, vias 0 -> 10
- net COL3: track 113.4 -> 211.3 mm, vias 10 -> 18
- net COL2: track 90.3 -> 178.4 mm, vias 8 -> 16
- net ROW8: track 216.6 -> 295.5 mm
- net ROW2: track 243.9 -> 308.3 mm, vias 0 -> 2
- net ROW4: track 248.7 -> 305.4 mm, vias 0 -> 2
- net ROW0: track 258.2 -> 303.2 mm, vias 0 -> 2
- net ROW6: track 265.5 -> 299.5 mm
- net COL6: track 212.7 -> 237.0 mm
- net Net-(D73-Pad2): track 0.00 -> 9.17 mm
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