File: HotSwap/Asok75hotswap.kicad_pcb (KiCad board)
At the start: 2 copper layers, 314.8 x 124.1 mm, 233 parts, among them J1 AVR-ISP-6, SW1 SW_Push, U1 PRTR5V0U2X, U2 ATmega32U4-MU, Y1 16MHz

Commit message: Routed underglow LEDs
Parts:
- moved R6 15.1 mm to (242.9, 115.1), turned to 180 degrees
- moved C11 9.38 mm to (153.3, 44.3), turned to 270 degrees
- moved C12 3.33 mm to (215.3, 44.3), turned to 270 degrees
- moved C5 2.30 mm to (-28.9, 147.8), turned to 180 degrees
- moved C10 2.00 mm to (91.4, 44.3), turned to 270 degrees
- moved C14 0.92 mm to (259.6, 113.9), turned to 270 degrees
- moved C13 0.90 mm to (259.6, 75.9), turned to 270 degrees
- moved C1 0.55 mm to (241.3, 152.2), turned to 180 degrees
- moved C6 0.52 mm to (-45.7, 115.7), turned to 90 degrees
- moved C7 0.51 mm to (-45.7, 77.7), turned to 90 degrees
- moved C4 0.26 mm to (64.5, 147.8), turned to 180 degrees
- moved C9 0.25 mm to (30.0, 44.3), turned to 270 degrees
- moved C8 0.23 mm to (-31.9, 44.3), turned to 270 degrees
- moved C3 0.22 mm to (134.8, 147.8), turned to 180 degrees
- moved C2 0.20 mm to (175.4, 147.8), turned to 180 degrees
- renumbered LED6 to LED10, LED8 to LED11, LED10 to LED12, LED12 to LED13, LED3 to LED2, LED5 to LED3, LED7 to LED4, LED9 to LED5, LED11 to LED6, LED13 to LED7, LED2 to LED8, LED4 to LED9
Connections:
- net LEDMOS renamed Net-(U2-Pad12)
- U2 pad 1: ROW0 -> Net-(U2-Pad1)
- U2 pad 10: LEDIND1 -> Net-(U2-Pad10)
- U2 pad 11: ROW1 -> Net-(U2-Pad11)
- U2 pad 18: RGBLED -> Net-(U2-Pad18)
- U2 pad 19: ROW11 -> Net-(U2-Pad19)
- U2 pad 20: ROW10 -> Net-(U2-Pad20)
- U2 pad 21: ROW8 -> Net-(U2-Pad21)
- U2 pad 22: ROW9 -> Net-(U2-Pad22)
- U2 pad 25: COL7 -> Net-(U2-Pad25)
- U2 pad 26: COL6 -> Net-(U2-Pad26)
- U2 pad 27: COL5 -> Net-(U2-Pad27)
- U2 pad 28: COL4 -> Net-(U2-Pad28)
- U2 pad 29: COL3 -> Net-(U2-Pad29)
- U2 pad 30: COL2 -> Net-(U2-Pad30)
- U2 pad 31: COL1 -> Net-(U2-Pad31)
- U2 pad 32: COL0 -> Net-(U2-Pad32)
- U2 pad 36: ROW7 -> Net-(U2-Pad36)
- U2 pad 37: ROW6 -> Net-(U2-Pad37)
- U2 pad 38: ROW5 -> Net-(U2-Pad38)
- U2 pad 39: ROW4 -> Net-(U2-Pad39)
- U2 pad 40: ROW3 -> Net-(U2-Pad40)
- U2 pad 41: ROW2 -> Net-(U2-Pad41)
- U2 pad 8: LEDIND3 -> Net-(U2-Pad8)
- U2 pad 9: LEDIND2 -> Net-(U2-Pad9)
Routing:
- net Net-(LED3-Pad3): track 0.00 -> 105.5 mm, vias 0 -> 4
- net Net-(LED4-Pad3): track 0.00 -> 103.9 mm, vias 0 -> 4
- net Net-(LED10-Pad3): track 0.00 -> 100.1 mm, vias 0 -> 2
- net Net-(LED6-Pad3): track 0.00 -> 96.0 mm, vias 0 -> 4
- net Net-(LED5-Pad3): track 0.00 -> 95.3 mm, vias 0 -> 4
- net Net-(LED11-Pad3): track 0.00 -> 77.7 mm, vias 0 -> 2
- net Net-(LED2-Pad3): track 0.00 -> 75.3 mm, vias 0 -> 6
- net Net-(LED13-Pad3): track 0.00 -> 73.1 mm, vias 0 -> 2
- net +5V: track 101.0 -> 162.1 mm, vias 7 -> 8
- net Net-(LED10-Pad1): track 0.00 -> 54.6 mm, vias 0 -> 2
- net Net-(LED7-Pad3): track 0.00 -> 54.3 mm, vias 0 -> 2
- net Net-(LED12-Pad3): track 0.00 -> 45.1 mm, vias 0 -> 2
- net Net-(LED8-Pad3): track 0.00 -> 42.7 mm, vias 0 -> 2
- net Net-(LED1-Pad3): track 0.00 -> 42.7 mm, vias 0 -> 2
- net GND: track 94.8 -> 136.6 mm
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
Commit message: Finished routing underglow LED power traces
Parts:
- moved SW1 11.9 mm to (240.3, 108.0), turned to 0 degrees
- moved R6 4.11 mm to (240.3, 111.9)
- moved R1 3.55 mm to (243.7, 48.4), turned to 90 degrees
- moved R2 3.55 mm to (243.7, 57.9), turned to 90 degrees
- moved R3 3.55 mm to (243.7, 67.5), turned to 90 degrees
- moved C19 3.17 mm to (234.9, 84.1)
- moved C17 2.38 mm to (234.9, 94.5)
- moved C21 2.38 mm to (233.4, 89.7)
- moved R9 2.38 mm to (244.5, 97.6)
- moved U2 2.38 mm to (240.3, 90.5)
- moved C15 2.38 mm to (244.3, 81.0)
- moved C16 2.38 mm to (236.2, 81.0)
- moved C18 2.38 mm to (245.6, 87.3)
- moved C20 2.38 mm to (244.5, 95.8)
- moved Y1 2.38 mm to (240.3, 81.0)
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Connections:
- J1 pad 1: ROW1 -> Net-(J1-Pad1)
- J1 pad 3: LEDIND2 -> Net-(J1-Pad3)
- J1 pad 4: LEDIND1 -> Net-(J1-Pad4)
- J1 pad 5: RESET -> Net-(J1-Pad5)
- U2 pad 18: Net-(U2-Pad18) -> LEDIND3
- U2 pad 19: Net-(U2-Pad19) -> LEDIND2
- U2 pad 20: Net-(U2-Pad20) -> LEDIND1
- U2 pad 21: Net-(U2-Pad21) -> COL7
Routing:
- net GND: track 136.6 -> 1191.5 mm, vias 2 -> 35
- net +5V: track 162.1 -> 1131.2 mm, vias 8 -> 35
- net RESET: track 2.19 -> 54.4 mm, vias 1 -> 3
- net LEDIND1: track 0.00 -> 50.0 mm, vias 0 -> 2
- net LEDIND2: track 0.00 -> 40.7 mm, vias 0 -> 2
- net LEDIND3: track 0.00 -> 30.9 mm, vias 0 -> 2
- net COL7: track 103.2 -> 116.9 mm
- net COL6: track 237.0 -> 249.4 mm
- net COL3: track 211.3 -> 221.9 mm
- net COL0: track 226.8 -> 235.5 mm
- net COL1: track 200.4 -> 208.0 mm
- net COL4: track 203.4 -> 211.0 mm
- net COL2: track 178.4 -> 185.1 mm
- net Net-(D86-Pad2): track 0.00 -> 5.50 mm, vias 0 -> 1
- net Net-(D84-Pad2): track 0.00 -> 5.50 mm, vias 0 -> 1
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