File: HotSwap/Old iterations/Asok75hotswap.kicad_pcb (KiCad board)
At the start: 2 copper layers, 321.9 x 124.1 mm, 349 parts, among them J1 AVR-ISP-6, Q1 2N7002, SW1 SW_Push, U1 ATmega32U4-MU, U2 PRTR5V0U2X, Y1 16MHz

Commit message: Updated hotswap PCB
Parts:
- moved LED9 77.2 mm to (-32.1, 40.5), turned to 0 degrees
- moved LED7 40.1 mm to (-48.4, 77.8), turned to 90 degrees
- moved LED8 38.0 mm to (-48.4, 115.7)
- moved LED14 1.60 mm to (241.1, 155.6)
- moved LED10 1.09 mm to (-28.9, 151.6)
- moved LED11 0.80 mm to (64.4, 151.6)
- moved LED6 0.71 mm to (29.8, 40.5)
- moved LED5 0.63 mm to (90.0, 40.5)
- moved LED12 0.63 mm to (134.6, 151.6)
- moved LED13 0.59 mm to (175.4, 151.6)
- moved LED2 0.39 mm to (262.7, 75.7)
- moved LED1 0.39 mm to (262.7, 114.1)
- moved LED4 0.39 mm to (159.4, 40.5)
- moved R6 0.38 mm to (244.5, 42.9)
- moved LED3 0.30 mm to (218.6, 40.5)
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Other:
- board size 321.9 x 124.1 mm -> 315.5 x 124.9 mm
