File: HotSwap/Old iterations/Asok75hotswapdone1.kicad_pcb (KiCad board)
At the start: 2 copper layers, 314.8 x 141 mm, 224 parts, among them J1 AVR-ISP-6, SW1 SW_Push, U1 ATmega32U4-MU, U2 PRTR5V0U2X, Y1 16MHz

Commit message: Finished routing hotswap version
Parts:
- moved C21 4.07 mm to (253.2, 151.4)
- moved RGB14 4.07 mm to (253.2, 154.8)
- moved MX_LEFT1 4.05 mm to (223.6, 148.2)
- moved D72 4.05 mm to (248.2, 133.9)
- moved D73 4.05 mm to (229.1, 153.0)
- moved D77 4.05 mm to (248.2, 153.0)
- moved D83 4.05 mm to (267.2, 153.0)
- moved Tab2 4.05 mm to (242.6, 156.1)
- moved MX_DOWN1 4.05 mm to (242.6, 148.2)
- moved MX_UP1 4.05 mm to (242.6, 129.2)
- moved MX_RIGHT1 4.05 mm to (261.7, 148.2)
- moved C2 4.05 mm to (257.5, 86.5)
- moved MX_DEL1 4.05 mm to (267.1, 47.6)
- moved MX_END1 4.05 mm to (267.1, 123.8)
- moved MX_HOME1 4.05 mm to (267.1, 66.7)
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Routing:
- net Net-(D72-Pad2): track 10.9 -> 9.23 mm
- net COL6: track 280.3 -> 281.8 mm
- net ROW8: track 361.6 -> 361.0 mm
- net ROW11: vias 6 -> 5
- removed copper zone on B.Cu, net GND
- removed copper zone on F.Cu, net GND
Other:
- outline, holes or cut-outs redrawn
- board text removed: "Designed by Asok"
- board text removed: "JLCJLCJLCJLC"
